Commit message: Add admittance controller (#3)
* update docs. re-parent robot arm to ground plane. Add force-torque sensor. update missing dependency

* add bridging from gz to ROS for force torque sensor

* add admittance controller

* added ros2_controls interface  for gazebo force torque sensor

* fix issues with sensor state_interface: We can't have 2 ros2_control tags, so we expand the ur_ros2_control xacro and insert the sensor tag into it.

* Update deps

Signed-off-by: Yadunund <yadunund@gmail.com>

* Cleanup readme

Signed-off-by: Yadunund <yadunund@gmail.com>

---------

Signed-off-by: Yadunund <yadunund@gmail.com>
Co-authored-by: JohnTGZ <johntangz@google.com>

File: ieec_description/urdf/ur_gz.urdf.xacro (robot description, xacro)
@@ -5,5 +5,6 @@
   <!-- import main macro -->
   <xacro:include filename="$(find ur_description)/urdf/ur_macro.xacro"/>
-  <xacro:include filename="$(find ur_simulation_gz)/urdf/ur_gz.ros2_control.xacro" />
+  <!-- <xacro:include filename="$(find ur_simulation_gz)/urdf/ur_gz.ros2_control.xacro" /> -->
+  <xacro:include filename="$(find ur_description)/urdf/inc/ur_joint_control.xacro" />
   <!-- possible 'ur_type' values: ur3, ur5, ur10, ur3e, ur5e, ur7e, ur10e, ur12e, ur16e, ur8long, ur15, ur20, ur30 -->
   <!-- the default value should raise an error in case this was called without defining the type -->
@@ -31,5 +32,5 @@
   <link name="world" />
   <link name="ground_plane">
-    <visual>
+    <!-- <visual>
       <origin rpy="0 0 0" xyz="0 0 0"/>
       <geometry>
@@ -39,5 +40,5 @@
         <color rgba="1 1 1 0.5"/>
       </material>
-    </visual>
+    </visual> -->
     <collision>
       <origin rpy="0 0 0" xyz="0 0 0"/>
@@ -56,5 +57,5 @@
     name="$(arg name)"
     tf_prefix="$(arg tf_prefix)"
-    parent="world"
+    parent="ground_plane"
     joint_limits_parameters_file="$(arg joint_limit_params)"
     kinematics_parameters_file="$(arg kinematics_params)"
@@ -77,10 +78,37 @@
       </ros>
     </plugin>
+    <plugin filename="gz-sim-forcetorque-system"
+            name="gz::sim::systems::ForceTorque">
+    </plugin>
+  </gazebo>
+  <gazebo reference="$(arg tf_prefix)wrist_3_joint">
+    <sensor name="force_torque_sensor" type="force_torque">
+      <always_on>true</always_on>
+      <update_rate>50</update_rate>
+      <visualize>true</visualize>
+      <topic>$(arg tf_prefix)wrist_3_joint/force_torque</topic>
+      <force_torque>
+        <frame>sensor</frame>
+        <measure_direction>parent_to_child</measure_direction>
+      </force_torque>
+    </sensor>
   </gazebo>
   <!-- ros2 control instance -->
-  <xacro:ur_ros2_control
-    name="$(arg name)"
-    tf_prefix="$(arg tf_prefix)"
-    transmission_hw_interface="$(arg transmission_hw_interface)"
-  />
+  <ros2_control name="GazeboSystem" type="system">
+    <hardware>
+      <plugin>gz_ros2_control/GazeboSimSystem</plugin>
+    </hardware>
+    <sensor name="force_torque_sensor" type="force_torque">
+      <state_interface name="force.x"/>
+      <state_interface name="force.y"/>
+      <state_interface name="force.z"/>
+      <state_interface name="torque.x"/>
+      <state_interface name="torque.y"/>
+      <state_interface name="torque.z"/>
+    </sensor>
+    <xacro:ur_joint_control_description
+      tf_prefix="$(arg tf_prefix)"
+      initial_positions="${dict(shoulder_pan_joint=0.0,shoulder_lift_joint=-1.57,elbow_joint=0.0,wrist_1_joint=-1.57,wrist_2_joint=0.0,wrist_3_joint=0.0)}"
+    />
+  </ros2_control>
 </robot>
