Commit message: Add and fix contact sensor (#14)
* add test block with pre-defined contact and friction parameters. Admittance Controller: Modified overdamping parameters and disable all axes except z-axis.

* change tool frame to tool0

* update documentation

* address review comments

* update size and mass of test block

* update readme

* Add and fix contact sensor.

* add back physics params

File: aic_assets/models/ATI_Axia80_M20/axia80_m20_macro.xacro (robot description, xacro)
@@ -4,5 +4,5 @@
   <xacro:property name="name" value="axia80_m20"/>
   <!-- TF prefix parameter -->
-  <xacro:property name="tf_prefix" value="ati"/>
+  <xacro:property name="tf_prefix" value="ati/"/>
   <!-- adapter_offset is the effective length that the adapter adds to the endeffector -->
   <xacro:property name="adapter_offset" value="0.0245"/>
@@ -106,5 +106,9 @@
       <sensor name="contact_sensor" type="contact">
         <contact>
-          <collision>collision1</collision>
+          <!-- The reason for the convoluted collision name reference is due to URDF to SDF
+          conversion prepending and appending names to the collision name. The current workaround
+          is provide an exact name -->
+          <collision>${tf_prefix}tool_link_fixed_joint_lump__collision1_collision</collision>
+          <topic>collision/tool_link</topic>
         </contact>
       </sensor>
