Commit message: Attach EOAT Assets to robot end-effector (#21)
* added models for eoat

* add urdf files and update ur_gz

* add urdf files and update ur_gz

* add gripper controller and state/command interfaces to gripper

* Build Gazebo Ionic from source (#11) (#24)

* update dependencies, repo and instructions to build gazebo ionic from source

* correct build instruction order

* update README

* update repos to use original packages instead of vendor

* Revert "update README"

This reverts commit c9f1cbff71e228795fc74065d534a2db6bed5319.

* Revert "update repos to use original packages instead of vendor"

This reverts commit d239a5466a78dc6cea13b26c45535bc37f6e686a.

* update readme and repo directories

* remove dartsim and ogre vendor packages

* Use tags for repo and update README



* update gz source packages in aic.repo and README.md for instructions to build from source and run from source

* update README and cmake dependencies for aic_gazebo

* update GZ_CONFIG_PATH directory in readme

* add environment hook for GZ_CONFIG_PATH, update gz vendor repo to use tags and update documentation

* Install gz deps via rosdep as well



* orge needs to be installed via gz deps



---------

Signed-off-by: JohnTGZ <johntangz@google.com>
Signed-off-by: Yadunund <yadunund@gmail.com>
Co-authored-by: John TGZ <johntangz@google.com>
Co-authored-by: Yadunund <yadunund@gmail.com>

* add gripper action and fix joint and mesh transforms. Added gazebo camera plugins. Change from ogre2 to ogre so that distortion can be rendered.

* add camera topics to gz_ros_bridge config

* Remove third wrist camera (#29)

* Adjust wrist camera params (#28)

* revert to ogre2 render_engine

---------

Signed-off-by: JohnTGZ <johntangz@google.com>
Signed-off-by: Yadunund <yadunund@gmail.com>
Co-authored-by: Cole Biesemeyer <cole.bsmr@gmail.com>
Co-authored-by: Morgan Quigley <morganquigley@intrinsic.ai>
Co-authored-by: Yadunund <yadunund@gmail.com>

File: aic_assets/models/Axia80 M20/axia80_m20_macro.xacro (robot description, xacro)
@@ -1,14 +1,12 @@
 <?xml version="1.0" ?>
 <robot xmlns:xacro="http://wiki.ros.org/xacro">
-  <!-- robot name parameter -->
-  <xacro:property name="name" value="axia80_m20"/>
   <!-- TF prefix parameter -->
   <xacro:property name="tf_prefix" value="ati/"/>
   <!-- adapter_offset is the effective length that the adapter adds to the endeffector -->
   <xacro:property name="adapter_offset" value="0.0245"/>
-  <xacro:macro name="axia80_m20" params="name tf_prefix">
+  <xacro:macro name="axia80_m20" params="tf_prefix">
     <link name="${tf_prefix}base_link">
       <inertial>
-        <origin xyz="0 0 ${adapter_offset / 2}" rpy="0 0 0"/>
+        <origin xyz="0 0 0" rpy="0 0 0"/>
         <mass value="0.36"/>
         <inertia ixx="0.0017389750000000002" ixy="0" ixz="0"
@@ -16,4 +14,22 @@
                  izz="0.0002521499999999999"/>
       </inertial>
+      <visual name="axia_ft_sensor_visual">
+        <origin xyz="0 0 0" rpy="0 0 0"/>
+        <geometry>
+          <mesh filename="package://aic_assets/models/Axia80 M20/axia_ft_sensor_visual.glb"/>
+        </geometry>
+      </visual>
+      <collision name="axia80_m20_collider_cylinder">
+        <origin xyz="0.0 -0.000004 0.012699" rpy="3.141593 0.0 0.0"/>
+        <geometry>
+          <cylinder length="0.025399" radius="0.041519"/>
+        </geometry>
+      </collision>
+      <collision name="axia80_m20001_collider_cylinder">
+        <origin xyz="0.0 0.041828 0.018432" rpy="-1.570796 0 0"/>
+        <geometry>
+          <cylinder radius="0.006027" length="0.016717"/>
+        </geometry>
+      </collision>
     </link>
     <joint name="${tf_prefix}attach_joint" type="fixed">
@@ -30,22 +46,4 @@
                  izz="0.000001"/>
       </inertial>
-      <visual>
-        <origin xyz="0 0 ${adapter_offset / 2}" rpy="0 0 0"/>
-        <geometry>
-          <cylinder length="${adapter_offset}" radius="0.041"/>
-        </geometry>
-      </visual>
-      <collision name="collision1">
-        <origin xyz="0 0 ${adapter_offset / 2}" rpy="0 0 0"/>
-        <geometry>
-          <cylinder length="${adapter_offset}" radius="0.041"/>
-        </geometry>
-      </collision>
-      <collision name="collision2">
-        <origin xyz="-0.0475 0 0.0075" rpy="0 0 0"/>
-        <geometry>
-          <box size="0.015 0.015 0.015"/>
-        </geometry>
-      </collision>
     </link>
     <gazebo reference="${tf_prefix}attach_joint">
@@ -103,21 +101,4 @@
       </sensor>
     </gazebo>
-    <gazebo reference="${tf_prefix}tool_link">
-      <sensor name="contact_sensor" type="contact">
-        <contact>
-          <!-- The reason for the convoluted collision name reference is due to URDF to SDF
-          conversion prepending and appending names to the collision name. The current workaround
-          is provide an exact name -->
-          <collision>${tf_prefix}tool_link_fixed_joint_lump__collision1_collision</collision>
-          <topic>collision/tool_link</topic>
-        </contact>
-      </sensor>
-      <!-- Reduce contact stiffness and damping for better stability -->
-      <kp>100000</kp>
-      <kd>100</kd>
-      <!-- Reduce friction in order to get smoother simulated force -->
-      <mu1>0.01</mu1>
-      <mu2>0.01</mu2>
-    </gazebo>
   </xacro:macro>
 </robot>

File: aic_description/urdf/ur_gz.urdf.xacro (robot description, xacro)
@@ -6,7 +6,11 @@
   <xacro:include filename="$(find ur_description)/urdf/ur_macro.xacro"/>
   <!-- import ATI Axia80-M20 macro -->
-  <xacro:include filename="$(find aic_assets)/models/ATI_Axia80_M20/axia80_m20_macro.xacro"/>
+  <xacro:include filename="$(find aic_assets)/models/Axia80 M20/axia80_m20_macro.xacro"/>
+  <xacro:include filename="$(find aic_assets)/models/Tri Cam Mount/tri_cam_mount_macro.xacro"/>
+  <xacro:include filename="$(find aic_assets)/models/Basler Camera/basler_camera_macro.xacro"/>
+  <xacro:include filename="$(find aic_assets)/models/Robotiq Hand-E/robotiq_hande_macro.xacro"/>
   <!-- <xacro:include filename="$(find ur_simulation_gz)/urdf/ur_gz.ros2_control.xacro" /> -->
   <xacro:include filename="$(find ur_description)/urdf/inc/ur_joint_control.xacro" />
+  <xacro:property name="D2R" value="${pi / 180.0}"/>
   <!-- possible 'ur_type' values: ur3, ur5, ur10, ur3e, ur5e, ur7e, ur10e, ur12e, ur16e, ur8long, ur15, ur20, ur30 -->
   <!-- the default value should raise an error in case this was called without defining the type -->
@@ -25,4 +29,12 @@
   <xacro:arg name="ros_namespace" default="" />
   <xacro:arg name="ati_tf_prefix" default="ati/" />
+  <xacro:arg name="cam_mount_tf_prefix" default="cam_mount/" />
+  <xacro:arg name="wrist_camera_1_tf_prefix" default="wrist_camera_1/"/>
+  <xacro:arg name="wrist_camera_2_tf_prefix" default="wrist_camera_2/"/>
+  <xacro:arg name="gripper_tf_prefix" default="gripper/"/>
+  <xacro:arg name="cam_lens_offset" default="0.035" />
+  <xacro:arg name="cam_mount_offset" default="0.09495" />
+  <!-- If true, enable Gazebo camera in sim -->
+  <xacro:arg name="use_sim_cam" default="${True}"/>
   <!-- Pose arguments for robot positioning -->
   <xacro:arg name="x" default="0.0" />
@@ -32,7 +44,4 @@
   <xacro:arg name="pitch" default="0.0" />
   <xacro:arg name="yaw" default="0.0" />
-  <xacro:property name="adapter_offset" value="0.0254"/>
-  <!-- <xacro:arg name="adapter_offset" default="0.0254" />
-  <xacro:arg name="adapter_offset_halved" default="0.0127" /> -->
   <!-- create link fixed to the "world" -->
   <link name="world" />
@@ -96,12 +105,62 @@
   <!-- ATI Force Torque sensor -->
   <xacro:axia80_m20
-    name="ati"
     tf_prefix="$(arg ati_tf_prefix)"
     >
   </xacro:axia80_m20>
+  <!-- Tri Cam Mount -->
+  <xacro:tri_cam_mount
+    tf_prefix="$(arg cam_mount_tf_prefix)"
+    >
+  </xacro:tri_cam_mount>
+  <xacro:basler_camera
+    name="wrist_camera_1"
+    tf_prefix="$(arg wrist_camera_1_tf_prefix)"
+    cam_lens_offset="$(arg cam_lens_offset)"
+    use_sim_cam="$(arg use_sim_cam)"
+    >
+  </xacro:basler_camera>
+  <xacro:basler_camera
+    name="wrist_camera_2"
+    tf_prefix="$(arg wrist_camera_2_tf_prefix)"
+    cam_lens_offset="$(arg cam_lens_offset)"
+    use_sim_cam="$(arg use_sim_cam)"
+    >
+  </xacro:basler_camera>
+  <xacro:robotiq_hande
+    name="gripper"
+    tf_prefix="$(arg gripper_tf_prefix)"
+    grip_pos_min="0.0"
+    grip_pos_max="0.025"
+    grip_vel_max="0.05"
+    grip_effort_max="130"
+    initial_pos="0.025"
+    >
+  </xacro:robotiq_hande>
+  <joint name="attach_tri_cam_mount" type="fixed">
+    <origin xyz="0 0 0" rpy="0 0 0"/>
+    <parent link="$(arg tf_prefix)tool0"/>
+    <child link="$(arg cam_mount_tf_prefix)cam_mount_link"/>
+  </joint>
   <joint name="attach_ft_sensor_joint" type="fixed">
-    <origin rpy="0 0 0" xyz="0 0 0"/>
-    <parent link="$(arg tf_prefix)tool0"/>
+    <origin xyz="0 0 0.0265" rpy="0 0 0"/>
+    <parent link="$(arg cam_mount_tf_prefix)cam_mount_link"/>
     <child link="$(arg ati_tf_prefix)base_link"/>
+  </joint>
+  <joint name="attach_wrist_camera_1" type="fixed">
+    <origin xyz="$(arg cam_mount_offset) 0 ${0.054483+$(arg cam_lens_offset)}"
+      rpy="0.261799 0 -1.5708"/>
+    <parent link="$(arg cam_mount_tf_prefix)cam_mount_link"/>
+    <child link="$(arg wrist_camera_1_tf_prefix)basler_cam_link"/>
+  </joint>
+  <joint name="attach_wrist_camera_2" type="fixed">
+    <origin xyz="-${$(arg cam_mount_offset) * sin(30.0*D2R)} -${$(arg cam_mount_offset) * cos(30.0*D2R)} ${0.054483+$(arg cam_lens_offset)}"
+      rpy="0.261799 0 2.61799"/>
+    <parent link="$(arg cam_mount_tf_prefix)cam_mount_link"/>
+    <child link="$(arg wrist_camera_2_tf_prefix)basler_cam_link"/>
+  </joint>
+  <joint name="attach_gripper" type="fixed">
+    <origin xyz="0 0 0" rpy="0 0 0"/>
+    <parent link="$(arg ati_tf_prefix)tool_link"/>
+    <child link="$(arg gripper_tf_prefix)hande_base_link"/>
   </joint>
   <!-- ros2 control instance -->
@@ -122,5 +181,5 @@
       initial_positions="${dict(
         shoulder_pan_joint=0.0,
-        shoulder_lift_joint=-1.8645,
+        shoulder_lift_joint=-1.2645,
         elbow_joint=-2.35,
         wrist_1_joint=-0.5,
