Commit message: Update parameters for Kilted distribution of ros2_controls: Update gripper action controller from position_controllers/GripperActionController to parallel_gripper_action_controller/GripperActionController. Add command_joints parameter for admittance_controller

File: aic_assets/models/Robotiq Hand-E/robotiq_hande.ros2_control.xacro (robot description, xacro)
@@ -1,5 +1,5 @@
 <?xml version="1.0"?>
 <robot xmlns:xacro="http://wiki.ros.org/xacro">
-  <xacro:macro name="robotiq_hande_ros2_control" params="name tf_prefix grip_pos_min grip_pos_max initial_pos">
+  <xacro:macro name="robotiq_hande_ros2_control" params="name tf_prefix grip_pos_min grip_pos_max grip_effort_min grip_effort_max initial_pos">
     <ros2_control name="${name}" type="system">
       <hardware>
@@ -11,4 +11,8 @@
           <param name="max">${grip_pos_max}</param>
         </command_interface>
+        <command_interface name="effort">
+          <param name="min">${grip_effort_min}</param>
+          <param name="max">${grip_effort_max}</param>
+        </command_interface>
         <state_interface name="position">
           <param name="initial_value">${initial_pos}</param>
@@ -17,4 +21,7 @@
           <param name="initial_value">0.0</param>
         </state_interface>
+        <state_interface name="effort">
+          <param name="initial_value">0.0</param>
+        </state_interface>
       </joint>
     </ros2_control>

File: aic_assets/models/Robotiq Hand-E/robotiq_hande_macro.xacro (robot description, xacro)
@@ -2,5 +2,5 @@
 <robot xmlns:xacro="http://wiki.ros.org/xacro">
   <xacro:include filename="$(find aic_assets)/models/Robotiq Hand-E/robotiq_hande.ros2_control.xacro"/>
-  <xacro:macro name="robotiq_hande" params="name tf_prefix grip_pos_min grip_pos_max grip_vel_max grip_effort_max initial_pos">
+  <xacro:macro name="robotiq_hande" params="name tf_prefix grip_pos_min grip_pos_max grip_vel_max grip_effort_min grip_effort_max initial_pos">
     <xacro:robotiq_hande_ros2_control
       name="${name}"
@@ -8,4 +8,6 @@
       grip_pos_min="${grip_pos_min}"
       grip_pos_max="${grip_pos_max}"
+      grip_effort_min="${grip_effort_min}"
+      grip_effort_max="${grip_effort_max}"
       initial_pos="${initial_pos}"
     />

File: aic_description/urdf/ur_gz.urdf.xacro (robot description, xacro)
@@ -133,4 +133,5 @@
     grip_pos_max="0.025"
     grip_vel_max="0.05"
+    grip_effort_min="20"
     grip_effort_max="130"
     initial_pos="0.025"

Commit message: Revert "Update parameters for Kilted distribution of ros2_controls: Update gripper action controller from position_controllers/GripperActionController to parallel_gripper_action_controller/GripperActionController. Add command_joints parameter for admittance_controller"
This reverts commit 0e29dc58590218db00907a0902ab068c506fa9e8.

File: aic_assets/models/Robotiq Hand-E/robotiq_hande.ros2_control.xacro (robot description, xacro)
@@ -1,5 +1,5 @@
 <?xml version="1.0"?>
 <robot xmlns:xacro="http://wiki.ros.org/xacro">
-  <xacro:macro name="robotiq_hande_ros2_control" params="name tf_prefix grip_pos_min grip_pos_max grip_effort_min grip_effort_max initial_pos">
+  <xacro:macro name="robotiq_hande_ros2_control" params="name tf_prefix grip_pos_min grip_pos_max initial_pos">
     <ros2_control name="${name}" type="system">
       <hardware>
@@ -11,8 +11,4 @@
           <param name="max">${grip_pos_max}</param>
         </command_interface>
-        <command_interface name="effort">
-          <param name="min">${grip_effort_min}</param>
-          <param name="max">${grip_effort_max}</param>
-        </command_interface>
         <state_interface name="position">
           <param name="initial_value">${initial_pos}</param>
@@ -21,7 +17,4 @@
           <param name="initial_value">0.0</param>
         </state_interface>
-        <state_interface name="effort">
-          <param name="initial_value">0.0</param>
-        </state_interface>
       </joint>
     </ros2_control>

File: aic_assets/models/Robotiq Hand-E/robotiq_hande_macro.xacro (robot description, xacro)
@@ -2,5 +2,5 @@
 <robot xmlns:xacro="http://wiki.ros.org/xacro">
   <xacro:include filename="$(find aic_assets)/models/Robotiq Hand-E/robotiq_hande.ros2_control.xacro"/>
-  <xacro:macro name="robotiq_hande" params="name tf_prefix grip_pos_min grip_pos_max grip_vel_max grip_effort_min grip_effort_max initial_pos">
+  <xacro:macro name="robotiq_hande" params="name tf_prefix grip_pos_min grip_pos_max grip_vel_max grip_effort_max initial_pos">
     <xacro:robotiq_hande_ros2_control
       name="${name}"
@@ -8,6 +8,4 @@
       grip_pos_min="${grip_pos_min}"
       grip_pos_max="${grip_pos_max}"
-      grip_effort_min="${grip_effort_min}"
-      grip_effort_max="${grip_effort_max}"
       initial_pos="${initial_pos}"
     />

File: aic_description/urdf/ur_gz.urdf.xacro (robot description, xacro)
@@ -133,5 +133,4 @@
     grip_pos_max="0.025"
     grip_vel_max="0.05"
-    grip_effort_min="20"
     grip_effort_max="130"
     initial_pos="0.025"
