Commit message: Update controls interface for kilted (#32)
* Update parameters for Kilted distribution of ros2_controls: Update gripper action controller from position_controllers/GripperActionController to parallel_gripper_action_controller/GripperActionController. Add command_joints parameter for admittance_controller

* fix path in GZ_SIM_RESOURCE_PATH hook

* fix GZ_SIM_RESOURCE_PATH hook by adding @CMAKE_INSTALL_PREFIX@/share/aic_assets/models

* Add runtime dependency on parallel_gripper_controller

* Offset visual and collision finger geometries (#33)

---------

Co-authored-by: Morgan Quigley <morganquigley@intrinsic.ai>

File: aic_assets/models/Robotiq Hand-E/robotiq_hande_macro.xacro (robot description, xacro)
@@ -2,5 +2,5 @@
 <robot xmlns:xacro="http://wiki.ros.org/xacro">
   <xacro:include filename="$(find aic_assets)/models/Robotiq Hand-E/robotiq_hande.ros2_control.xacro"/>
-  <xacro:macro name="robotiq_hande" params="name tf_prefix grip_pos_min grip_pos_max grip_vel_max grip_effort_max initial_pos">
+  <xacro:macro name="robotiq_hande" params="name tf_prefix grip_pos_min grip_pos_max grip_vel_max grip_effort_min grip_effort_max initial_pos">
     <xacro:robotiq_hande_ros2_control
       name="${name}"
@@ -8,6 +8,9 @@
       grip_pos_min="${grip_pos_min}"
       grip_pos_max="${grip_pos_max}"
+      grip_effort_min="${grip_effort_min}"
+      grip_effort_max="${grip_effort_max}"
       initial_pos="${initial_pos}"
     />
+    <xacro:property name="gripper_jaw_offset" value="0.025"/>
     <link name="${tf_prefix}hande_base_link">
       <inertial>
@@ -46,5 +49,5 @@
       </inertial>
       <visual name="hande_finger_visual">
-        <origin xyz="0 0 0" rpy="0 0 0"/>
+        <origin xyz="${-gripper_jaw_offset} 0 0" rpy="0 0 0"/>
         <geometry>
           <mesh filename="package://aic_assets/models/Robotiq Hand-E/hande_finger_visual.glb"/>
@@ -52,5 +55,5 @@
       </visual>
       <collision name="finger_collider_box">
-        <origin xyz="0.032595 -0.00001 0.138138" rpy="0.0 0.0 0.0"/>
+        <origin xyz="${-gripper_jaw_offset + 0.032595} -0.00001 0.138138" rpy="0.0 0.0 0.0"/>
         <geometry>
           <box size="0.007839 0.021 0.028622"/>
@@ -58,5 +61,5 @@
       </collision>
       <collision name="finger_collider_box001">
-        <origin xyz="0.028 -0.00001 0.16145" rpy="0.0 0.0 0.0"/>
+        <origin xyz="${-gripper_jaw_offset + 0.028} -0.00001 0.16145" rpy="0.0 0.0 0.0"/>
         <geometry>
           <box size="0.006 0.021 0.021498"/>
@@ -64,5 +67,5 @@
       </collision>
       <collision name="finger_collider_box002">
-        <origin xyz="0.014354 -0.015 0.124725" rpy="0.0 0.0 0.0"/>
+        <origin xyz="${-gripper_jaw_offset + 0.014354} -0.015 0.124725" rpy="0.0 0.0 0.0"/>
         <geometry>
           <box size="0.044319 0.0075 0.003949"/>
@@ -70,5 +73,5 @@
       </collision>
       <collision name="finger_collider_box003">
-        <origin xyz="0.027046 -0.00954 0.129064" rpy="0.0 0.0 0.0"/>
+        <origin xyz="${-gripper_jaw_offset + 0.027046} -0.00954 0.129064" rpy="0.0 0.0 0.0"/>
         <geometry>
           <box size="0.017387 0.018419 0.009271"/>
@@ -90,5 +93,5 @@
       </inertial>
       <visual name="hande_finger_visual">
-        <origin xyz="0 0 0" rpy="0 0 3.14157"/>
+        <origin xyz="${gripper_jaw_offset} 0 0" rpy="0 0 3.14157"/>
         <geometry>
           <mesh filename="package://aic_assets/models/Robotiq Hand-E/hande_finger_visual.glb"/>
@@ -96,5 +99,5 @@
       </visual>
       <collision name="finger_collider_box">
-        <origin xyz="-0.032595 -0.00001 0.138138" rpy="0.0 0.0 0.0"/>
+        <origin xyz="${gripper_jaw_offset - 0.032595} -0.00001 0.138138" rpy="0.0 0.0 0.0"/>
         <geometry>
           <box size="0.007839 0.021 0.028622"/>
@@ -102,5 +105,5 @@
       </collision>
       <collision name="finger_collider_box001">
-        <origin xyz="-0.028 -0.00001 0.16145" rpy="0.0 0.0 0.0"/>
+        <origin xyz="${gripper_jaw_offset - 0.028} -0.00001 0.16145" rpy="0.0 0.0 0.0"/>
         <geometry>
           <box size="0.006 0.021 0.021498"/>
@@ -108,5 +111,5 @@
       </collision>
       <collision name="finger_collider_box002">
-        <origin xyz="-0.014354 -0.015 0.124725" rpy="0.0 0.0 0.0"/>
+        <origin xyz="${gripper_jaw_offset - 0.014354} -0.015 0.124725" rpy="0.0 0.0 0.0"/>
         <geometry>
           <box size="0.044319 0.0075 0.003949"/>
@@ -114,5 +117,5 @@
       </collision>
       <collision name="finger_collider_box003">
-        <origin xyz="-0.027046 -0.00954 0.129064" rpy="0.0 0.0 0.0"/>
+        <origin xyz="${gripper_jaw_offset - 0.027046} -0.00954 0.129064" rpy="0.0 0.0 0.0"/>
         <geometry>
           <box size="0.017387 0.018419 0.009271"/>
@@ -142,5 +145,5 @@
     <link name="${tf_prefix}tool_frame"/>
     <joint name="${tf_prefix}attach_tool_frame" type="fixed">
-      <origin xyz="0 0 0.128" rpy="0 0 0"/>
+      <origin xyz="0 0 0.172" rpy="0 0 0"/>
       <parent link="${tf_prefix}hande_base_link"/>
       <child link="${tf_prefix}tool_frame"/>

File: aic_description/urdf/ur_gz.urdf.xacro (robot description, xacro)
@@ -133,6 +133,7 @@
     grip_pos_max="0.025"
     grip_vel_max="0.05"
+    grip_effort_min="20"
     grip_effort_max="130"
-    initial_pos="0.025"
+    initial_pos="0.02"
     >
   </xacro:robotiq_hande>

Commit message: update frame names

File: aic_assets/models/Robotiq Hand-E/robotiq_hande_macro.xacro (robot description, xacro)
@@ -143,9 +143,9 @@
       <mimic joint="${tf_prefix}left_finger_joint" multiplier="1" offset="0"/>
     </joint>
-    <link name="${tf_prefix}tool_frame"/>
+    <link name="${tf_prefix}tcp"/>
     <joint name="${tf_prefix}attach_tool_frame" type="fixed">
       <origin xyz="0 0 0.172" rpy="0 0 0"/>
       <parent link="${tf_prefix}hande_base_link"/>
-      <child link="${tf_prefix}tool_frame"/>
+      <child link="${tf_prefix}tcp"/>
     </joint>
   </xacro:macro>
