Commit message: change tri cam mount naming to cam mount. remove unused wrist_camera_3 gz_ros_bridge topic. (#30)

File: aic_assets/models/Camera Mount/cam_mount_macro.xacro (robot description, xacro)
@@ -2,5 +2,5 @@
 <robot xmlns:xacro="http://wiki.ros.org/xacro">
   <xacro:property name="tf_prefix" value="cam_mount/"/>
-  <xacro:macro name="tri_cam_mount" params="tf_prefix">
+  <xacro:macro name="camera_mount" params="tf_prefix">
     <link name="${tf_prefix}cam_mount_link">
       <inertial>
@@ -13,5 +13,5 @@
       <visual name="cam_mount_visual">
         <geometry>
-          <mesh filename="package://aic_assets/models/Tri Cam Mount/cam_mount_visual.glb"/>
+          <mesh filename="package://aic_assets/models/Camera Mount/cam_mount_visual.glb"/>
         </geometry>
       </visual>

File: aic_description/urdf/ur_gz.urdf.xacro (robot description, xacro)
@@ -7,5 +7,5 @@
   <!-- import ATI Axia80-M20 macro -->
   <xacro:include filename="$(find aic_assets)/models/Axia80 M20/axia80_m20_macro.xacro"/>
-  <xacro:include filename="$(find aic_assets)/models/Tri Cam Mount/tri_cam_mount_macro.xacro"/>
+  <xacro:include filename="$(find aic_assets)/models/Camera Mount/cam_mount_macro.xacro"/>
   <xacro:include filename="$(find aic_assets)/models/Basler Camera/basler_camera_macro.xacro"/>
   <xacro:include filename="$(find aic_assets)/models/Robotiq Hand-E/robotiq_hande_macro.xacro"/>
@@ -108,9 +108,9 @@
     >
   </xacro:axia80_m20>
-  <!-- Tri Cam Mount -->
-  <xacro:tri_cam_mount
+  <!-- Camera Mount -->
+  <xacro:camera_mount
     tf_prefix="$(arg cam_mount_tf_prefix)"
     >
-  </xacro:tri_cam_mount>
+  </xacro:camera_mount>
   <xacro:basler_camera
     name="wrist_camera_1"
@@ -137,5 +137,5 @@
     >
   </xacro:robotiq_hande>
-  <joint name="attach_tri_cam_mount" type="fixed">
+  <joint name="attach_cam_mount" type="fixed">
     <origin xyz="0 0 0" rpy="0 0 0"/>
     <parent link="$(arg tf_prefix)tool0"/>

Commit message: Use three wrist cameras, at 60 degree intervals

File: aic_assets/models/Camera Mount/cam_mount_macro.xacro (robot description, xacro)
@@ -14,4 +14,10 @@
       <visual name="cam_mount_visual">
         <origin xyz="0.0 0.0 0.0215" rpy="0.0 0.0 ${z_rot}"/>
+        <geometry>
+          <mesh filename="package://aic_assets/models/Camera Mount/cam_mount_visual.glb"/>
+        </geometry>
+      </visual>
+      <visual name="cam_mount_visual_repeated">
+        <origin xyz="0.0 0.0 0.0215" rpy="0.0 0.0 ${z_rot + 3.1415926}"/>
         <geometry>
           <mesh filename="package://aic_assets/models/Camera Mount/cam_mount_visual.glb"/>

File: aic_description/urdf/ur_gz.urdf.xacro (robot description, xacro)
@@ -32,4 +32,5 @@
   <xacro:arg name="wrist_camera_1_tf_prefix" default="wrist_camera_1/"/>
   <xacro:arg name="wrist_camera_2_tf_prefix" default="wrist_camera_2/"/>
+  <xacro:arg name="wrist_camera_3_tf_prefix" default="wrist_camera_3/"/>
   <xacro:arg name="gripper_tf_prefix" default="gripper/"/>
   <xacro:arg name="cam_mount_radial_offset" default="0.1" />
@@ -125,4 +126,10 @@
     >
   </xacro:basler_camera>
+  <xacro:basler_camera
+    name="wrist_camera_3"
+    tf_prefix="$(arg wrist_camera_3_tf_prefix)"
+    use_sim_cam="$(arg use_sim_cam)"
+    >
+  </xacro:basler_camera>
   <xacro:robotiq_hande
     name="gripper"
@@ -136,4 +143,7 @@
     >
   </xacro:robotiq_hande>
+ <!-- ********************
+      ** wrist_camera_1 **
+      ******************** -->
   <joint name="attach_cam_mount" type="fixed">
     <origin xyz="0 0 -.0265" rpy="0 0 0"/>
@@ -157,6 +167,6 @@
   </link>
   <joint name="wrist_camera_1_intermediate_joint" type="fixed">
-    <origin xyz="0 -$(arg cam_mount_radial_offset) $(arg cam_mount_axial_offset)"
-      rpy="${90.0*D2R} ${-90.0*D2R} ${0.0*D2R}"/>
+    <origin xyz="${-cos(30.0*D2R)*$(arg cam_mount_radial_offset)} -${sin(30.0*D2R)*$(arg cam_mount_radial_offset)} $(arg cam_mount_axial_offset)"
+      rpy="${90.0*D2R} ${-90.0*D2R} ${-60.0*D2R}"/>
     <parent link="$(arg cam_mount_tf_prefix)cam_mount_link"/>
     <child link="wrist_camera_1_intermediate_link"/>
@@ -167,4 +177,7 @@
     <child link="$(arg wrist_camera_1_tf_prefix)basler_cam_link"/>
   </joint>
+  <!-- ********************
+       ** wrist_camera_2 **
+       ******************** -->
   <!-- Dummy link to simplify the chain of rotations -->
   <link name="wrist_camera_2_intermediate_link">
@@ -178,6 +191,6 @@
   </link>
   <joint name="wrist_camera_2_intermediate_joint" type="fixed">
-    <origin xyz="${-cos(30.0*D2R)*$(arg cam_mount_radial_offset)} ${sin(30.0*D2R)*$(arg cam_mount_radial_offset)} $(arg cam_mount_axial_offset)"
-      rpy="${90.0*D2R} ${-90.0*D2R} ${-120.0*D2R}"/>
+    <origin xyz="0 -$(arg cam_mount_radial_offset) $(arg cam_mount_axial_offset)"
+      rpy="${90.0*D2R} ${-90.0*D2R} ${0.0*D2R}"/>
     <parent link="$(arg cam_mount_tf_prefix)cam_mount_link"/>
     <child link="wrist_camera_2_intermediate_link"/>
@@ -187,4 +200,28 @@
     <parent link="wrist_camera_2_intermediate_link"/>
     <child link="$(arg wrist_camera_2_tf_prefix)basler_cam_link"/>
+  </joint>
+  <!-- ********************
+       ** wrist_camera_3 **
+       ******************** -->
+  <!-- Dummy link to simplify the chain of rotations -->
+  <link name="wrist_camera_3_intermediate_link">
+    <inertial>
+      <origin xyz="0 0 0" rpy="0 0 0"/>
+      <mass value="0.001"/>
+      <inertia ixx="0.000001" ixy="0" ixz="0"
+               iyy="0.000001" iyz="0"
+               izz="0.000001"/>
+    </inertial>
+  </link>
+  <joint name="wrist_camera_3_intermediate_joint" type="fixed">
+    <origin xyz="${cos(30.0*D2R)*$(arg cam_mount_radial_offset)} -${sin(30.0*D2R)*$(arg cam_mount_radial_offset)} $(arg cam_mount_axial_offset)"
+      rpy="${90.0*D2R} ${-90.0*D2R} ${60.0*D2R}"/>
+    <parent link="$(arg cam_mount_tf_prefix)cam_mount_link"/>
+    <child link="wrist_camera_3_intermediate_link"/>
+  </joint>
+  <joint name="attach_wrist_camera_3" type="fixed">
+    <origin xyz="0 0 0" rpy="${0.0*D2R} ${15.0*D2R} ${0.0*D2R}"/>
+    <parent link="wrist_camera_3_intermediate_link"/>
+    <child link="$(arg wrist_camera_3_tf_prefix)basler_cam_link"/>
   </joint>
   <joint name="attach_gripper" type="fixed">

Commit message: update cam_mount xacro

File: aic_assets/models/Camera Mount/cam_mount_macro.xacro (robot description, xacro)
@@ -13,14 +13,4 @@
       </inertial>
       <visual name="cam_mount_visual">
-        <origin xyz="0.0 0.0 0.0215" rpy="0.0 0.0 ${z_rot}"/>
-        <geometry>
-          <mesh filename="package://aic_assets/models/Camera Mount/cam_mount_visual.glb"/>
-        </geometry>
-      </visual>
-      <!-- TODO(anyone): Update the camera mount visual to have arms at [-60, 0, +60].
-           The repeated camera mount is just a placeholder, and it adds "extra" arms
-           arms that we are not currently using, since we have 3 cameras, not 6. -->
-      <visual name="cam_mount_visual_repeated">
-        <origin xyz="0.0 0.0 0.0215" rpy="0.0 0.0 ${z_rot + 3.1415926}"/>
         <geometry>
           <mesh filename="package://aic_assets/models/Camera Mount/cam_mount_visual.glb"/>
@@ -28,5 +18,5 @@
       </visual>
       <collision name="cam_mount_collider_cylinder">
-        <origin xyz="0.0 0.0 0.0215" rpy="0.0 0.0 ${z_rot}"/>
+        <origin xyz="0.0 0.0 0.0215" rpy="0.0 0.0 0.0"/>
         <geometry>
           <cylinder radius="0.06" length="0.01"/>
@@ -34,5 +24,5 @@
       </collision>
       <collision name="cam_mount_collider_cylinder.001">
-        <origin xyz="0.0 0.0 0.012638" rpy="0.0 0.0 ${z_rot}"/>
+        <origin xyz="0.0 0.0 0.012638" rpy="0.0 0.0 0.0"/>
         <geometry>
           <cylinder radius="0.030383" length="0.025275"/>
@@ -41,37 +31,55 @@
       <!-- TODO(anyone): Update the colliders to match the [-60, 0, +60] cameras. -->
       <collision name="cam_mount003_collider_box">
-        <origin xyz="0.068974 0.000189 0.02" rpy="0.0 0.0 ${z_rot}"/>
+        <origin xyz="0.000252 -0.068974 0.0193" rpy="0.0 0.0 -1.570796"/>
         <geometry>
-          <box size="0.055675 0.027622 0.003"/>
+          <box size="0.055675 0.036898 0.0044"/>
         </geometry>
       </collision>
       <collision name="cam_mount003_collider_box.001">
-        <origin xyz="0.096142 0.000189 0.021981" rpy="0.0 1.308997 ${z_rot}"/>
+        <origin xyz="0.000189 -0.100267 0.003926" rpy="0.0 1.308997 -1.570796"/>
         <geometry>
-          <box size="0.035256 0.027622 0.003"/>
+          <box size="0.035256 0.04325 0.00858"/>
         </geometry>
       </collision>
       <collision name="cam_mount003_collider_box.002">
-        <origin xyz="-0.034323 -0.059827 0.02" rpy="0.0 0.0 ${z_rot - 2.094395}"/>
+        <origin xyz="0.000252 -0.076575 0.007442" rpy="0.0 0.479966 -1.570796"/>
         <geometry>
-          <box size="0.055675 0.027622 0.003"/>
+          <box size="0.059567 0.036898 0.010442"/>
         </geometry>
       </collision>
       <collision name="cam_mount003_collider_box.003">
-        <origin xyz="-0.047908 -0.083356 0.021981" rpy="0.0 1.308997 ${z_rot - 2.094395}"/>
+        <origin xyz="0.059859 -0.034268 0.0193" rpy="0.0 0.0 -0.523599"/>
         <geometry>
-          <box size="0.035256 0.027622 0.003"/>
+          <box size="0.055675 0.036898 0.0044"/>
         </geometry>
       </collision>
       <collision name="cam_mount003_collider_box.004">
-        <origin xyz="-0.03465 0.059639 0.02" rpy="0.0 0.0 ${z_rot - 4.18879}"/>
+        <origin xyz="0.086928 -0.04997 0.003926" rpy="0.0 1.308997 -0.523599"/>
         <geometry>
-          <box size="0.055675 0.027622 0.003"/>
+          <box size="0.035256 0.04325 0.00858"/>
         </geometry>
       </collision>
       <collision name="cam_mount003_collider_box.005">
-        <origin xyz="-0.048235 0.083167 0.021981" rpy="0.0 1.308997 ${z_rot - 4.18879}"/>
+        <origin xyz="0.06619 -0.037924 0.007593" rpy="0.0 0.479965 -0.523599"/>
         <geometry>
-          <box size="0.035256 0.027622 0.003"/>
+          <box size="0.060221 0.036898 0.010442"/>
+        </geometry>
+      </collision>
+      <collision name="cam_mount003_collider_box.006">
+        <origin xyz="-0.059607 -0.034705 0.0193" rpy="0.0 -0.0 -2.617994"/>
+        <geometry>
+          <box size="0.055675 0.036898 0.0044"/>
+        </geometry>
+      </collision>
+      <collision name="cam_mount003_collider_box.007">
+        <origin xyz="-0.08674 -0.050297 0.003926" rpy="0.0 1.308997 -2.617994"/>
+        <geometry>
+          <box size="0.035256 0.04325 0.00858"/>
+        </geometry>
+      </collision>
+      <collision name="cam_mount003_collider_box.008">
+        <origin xyz="-0.066139 -0.038476 0.007473" rpy="0.0 0.479965 -2.617994"/>
+        <geometry>
+          <box size="0.0597 0.036898 0.010442"/>
         </geometry>
       </collision>

Commit message: remove unused z_rot

File: aic_assets/models/Camera Mount/cam_mount_macro.xacro (robot description, xacro)
@@ -2,5 +2,4 @@
 <robot xmlns:xacro="http://wiki.ros.org/xacro">
   <xacro:property name="tf_prefix" value="cam_mount/"/>
-  <xacro:property name="z_rot" value="-1.57079"/>
   <xacro:macro name="camera_mount" params="tf_prefix">
     <link name="${tf_prefix}cam_mount_link">
