Commit message: update sc port, nic card mount, and task board collisions (#72)
Signed-off-by: Ian Chen <ichen@openrobotics.org>

File: aic_assets/models/NIC Card Mount/nic_card_mount_macro.xacro (robot description, xacro)
@@ -95,4 +95,88 @@
         </geometry>
       </collision>
+      <collision name="10099100-011lfc001_collider_box">
+        <origin xyz="-0.017799 -0.052954 0.00548" rpy="3.128092 0.0 0.0"/>
+        <geometry>
+          <box size="0.001099 0.04872 0.011083"/>
+        </geometry>
+      </collision>
+      <collision name="10099100-011lfc001_collider_box.001">
+        <origin xyz="-0.002687 -0.052954 0.005461" rpy="3.128092 0.0 0.0"/>
+        <geometry>
+          <box size="0.001125 0.04872 0.011121"/>
+        </geometry>
+      </collision>
+      <collision name="10099100-011lfc001_collider_box.002">
+        <origin xyz="-0.010237 -0.052889 0.010234" rpy="3.128092 0.0 0.0"/>
+        <geometry>
+          <box size="0.016224 0.04872 0.000923"/>
+        </geometry>
+      </collision>
+      <collision name="10099100-011lfc001_collider_box.003">
+        <origin xyz="-0.010237 -0.053024 0.000296" rpy="3.128092 0.0 0.0"/>
+        <geometry>
+          <box size="0.016224 0.04872 0.001054"/>
+        </geometry>
+      </collision>
+      <collision name="10099100-011lfc001_collider_box.004">
+        <origin xyz="-0.010237 -0.028738 0.003845" rpy="3.128092 0.0 0.0"/>
+        <geometry>
+          <box size="0.016224 0.00025 0.013698"/>
+        </geometry>
+      </collision>
+      <collision name="10099100-011lfc001_collider_box.005">
+        <origin xyz="0.005401 -0.052954 0.00548" rpy="3.128092 0.0 0.0"/>
+        <geometry>
+          <box size="0.001099 0.04872 0.011083"/>
+        </geometry>
+      </collision>
+      <collision name="10099100-011lfc001_collider_box.006">
+        <origin xyz="0.020513 -0.052954 0.005461" rpy="3.128092 0.0 0.0"/>
+        <geometry>
+          <box size="0.001125 0.04872 0.011121"/>
+        </geometry>
+      </collision>
+      <collision name="10099100-011lfc001_collider_box.007">
+        <origin xyz="0.012963 -0.052889 0.010234" rpy="3.128092 0.0 0.0"/>
+        <geometry>
+          <box size="0.016224 0.04872 0.00092"/>
+        </geometry>
+      </collision>
+      <collision name="10099100-011lfc001_collider_box.008">
+        <origin xyz="0.012963 -0.053024 0.000296" rpy="3.128092 0.0 0.0"/>
+        <geometry>
+          <box size="0.016224 0.04872 0.001054"/>
+        </geometry>
+      </collision>
+      <collision name="10099100-011lfc001_collider_box.009">
+        <origin xyz="0.012963 -0.028738 0.003845" rpy="3.128092 0.0 0.0"/>
+        <geometry>
+          <box size="0.016224 0.00025 0.01369"/>
+        </geometry>
+      </collision>
+      <collision name="plane001_collider_box">
+        <origin xyz="-0.007649 -0.074646 -0.0007515" rpy="0.0 0.0 0.0"/>
+        <geometry>
+          <box size="0.113402 0.000875 0.003449"/>
+        </geometry>
+      </collision>
+      <collision name="plane001_collider_box.001">
+        <origin xyz="-0.007649 -0.074646 0.01352" rpy="0.0 0.0 0.0"/>
+        <geometry>
+          <box size="0.113402 0.000875 0.00501"/>
+        </geometry>
+      </collision>
+      <collision name="plane001_collider_box.002">
+        <origin xyz="0.038559 -0.074646 0.006455" rpy="0.0 0.0 0.0"/>
+        <geometry>
+          <box size="0.036181 0.000875 0.01112"/>
+        </geometry>
+      </collision>
+      <collision name="plane001_collider_box.003">
+        <origin xyz="-0.041261 -0.074646 0.006455" rpy="0.0 0.0 0.0"/>
+        <geometry>
+          <box size="0.046178 0.000875 0.011123"/>
+        </geometry>
+      </collision>
     </link>
     <!-- Joint connecting card to mount -->

File: aic_assets/models/SC Port/sc_port_macro.xacro (robot description, xacro)
@@ -23,5 +23,23 @@
         <origin xyz="0.0 0.0 0.004225" rpy="0.0 0.0 0.0"/>
         <geometry>
-          <box size="0.025781 0.027432 0.00085"/>
+          <box size="0.025781 0.0108 0.00085"/>
+        </geometry>
+      </collision>
+      <collision name="cube_collider_box_mid">
+        <origin xyz="0.0 0.0 0.004225" rpy="0.0 0.0 0.0"/>
+        <geometry>
+          <box size="0.0103 0.027432 0.00085"/>
+        </geometry>
+      </collision>
+      <collision name="cube_collider_box_mid02">
+        <origin xyz="0.01 0.0 0.004225" rpy="0.0 0.0 0.0"/>
+        <geometry>
+          <box size="0.005 0.027432 0.00085"/>
+        </geometry>
+      </collision>
+      <collision name="cube_collider_box_mid03">
+        <origin xyz="-0.01 0.0 0.004225" rpy="0.0 0.0 0.0"/>
+        <geometry>
+          <box size="0.005 0.027432 0.00085"/>
         </geometry>
       </collision>
@@ -56,10 +74,4 @@
         </geometry>
       </collision>
-      <collision name="foa_005a_3d_collider_box">
-        <origin xyz="0.0 0.0 0.0" rpy="3.141593 0.0 0.0"/>
-        <geometry>
-          <box size="0.025 0.002946 0.009"/>
-        </geometry>
-      </collision>
     </link>
   </xacro:macro>

File: aic_assets/models/Task Board Base/task_board_base_macro.xacro (robot description, xacro)
@@ -14,14 +14,33 @@
         </geometry>
       </visual>
-      <collision name="v1015074_collider_box">
-        <origin xyz="-0.075 0.05 0.0105" rpy="0.0 0.0 0.0"/>
+      <collision name="v1015083001_collider_box_left">
+        <origin xyz="0.0 -0.10 0.0075" rpy="0.0 0.0 0.0"/>
         <geometry>
-          <box size="0.14 0.087 0.005"/>
+          <box size="0.3 0.228 0.005"/>
         </geometry>
       </collision>
-      <collision name="v1015083001_collider_box">
-        <origin xyz="0.0 0.0 0.0075" rpy="0.0 0.0 0.0"/>
+      <collision name="v1015083001_collider_right">
+        <origin xyz="0.0 0.149 0.0075" rpy="0.0 0.0 0.0"/>
         <geometry>
-          <box size="0.3 0.425 0.005"/>
+          <box size="0.3 0.127 0.005"/>
+        </geometry>
+      </collision>
+      <collision name="v1015083001_collider_mid">
+        <pose>0.0 0.0 -0.0</pose>
+        <origin xyz="-0.075 0.05 0.0075" rpy="0.0 0.0 0.0"/>
+        <geometry>
+          <box size="0.14 0.012 0.005"/>
+        </geometry>
+      </collision>
+      <collision name="v1015083001_collider_bottom">
+        <origin xyz="0.068 0.0 0.0075" rpy="0.0 0.0 0.0"/>
+        <geometry>
+          <box size="0.165 0.425 0.005"/>
+        </geometry>
+      </collision>
+      <collision name="v1015083001_collider_top">
+        <origin xyz="-0.143 0.0 0.0075" rpy="0.0 0.0 0.0"/>
+        <geometry>
+          <box size="0.015 0.425 0.005"/>
         </geometry>
       </collision>

Commit message: Added SFP dummy links (#74)
* added sfp dummy links

* Rename frames to match convention and add them to NIC Mount

Signed-off-by: Yadunund <yadunund@intrinsic.ai>

---------

Signed-off-by: Yadunund <yadunund@intrinsic.ai>
Co-authored-by: Yadunund <yadunund@intrinsic.ai>

File: aic_assets/models/NIC Card Mount/nic_card_mount_macro.xacro (robot description, xacro)
@@ -186,4 +186,18 @@
       <origin xyz="0 -0.01785 0.0799" rpy="-1.57 0 0"/>
     </joint>
+    <!-- SFP Port 0 Link -->
+    <link name="${prefix}sfp_port_0_link"/>
+    <joint name="${prefix}sfp_port_0_joint" type="fixed">
+      <parent link="${prefix}card_link"/>
+      <child link="${prefix}sfp_port_0_link"/>
+      <origin xyz="0.01295 -0.031572 0.00501" rpy="4.69895 0 0"/>
+    </joint>
+    <!-- SFP Port 1 Link -->
+    <link name="${prefix}sfp_port_1_link"/>
+    <joint name="${prefix}sfp_port_1_joint" type="fixed">
+      <parent link="${prefix}card_link"/>
+      <child link="${prefix}sfp_port_1_link"/>
+      <origin xyz="-0.01025 -0.031572 0.00501" rpy="4.69895 0 0"/>
+    </joint>
   </xacro:macro>
 </robot>
