Commit message: Detect SC and SFP plug-port insertion (#77)
* update sc port, nic card mount, and task board collisions

Signed-off-by: Ian Chen <ichen@openrobotics.org>

* replace sfp and nic card mount urdf with gazebo include tag

Signed-off-by: Ian Chen <ichen@openrobotics.org>

* Add contact collision and touch plugin

Signed-off-by: Ian Chen <ichen@openrobotics.org>

* use custom gz-physics branch

Signed-off-by: Ian Chen <ichen@openrobotics.org>

* Add the visual representation of the AIC board

* Delete docs/taskboard.webp

Sorry for commit directly to main...

* update cam near far clip plane so we can zoom in to see small details

Signed-off-by: Ian Chen <ichen@openrobotics.org>

* Lock cable in place after insertion (#80)

* Extend cable plugin to lock cables in place

Signed-off-by: Ian Chen <ichen@openrobotics.org>

* lint

Signed-off-by: Ian Chen <ichen@openrobotics.org>

* more lint

Signed-off-by: Ian Chen <ichen@openrobotics.org>

* remove empty line:

Signed-off-by: Ian Chen <ichen@openrobotics.org>

---------

Signed-off-by: Ian Chen <ichen@openrobotics.org>

---------

Signed-off-by: Ian Chen <ichen@openrobotics.org>
Co-authored-by: jimmybaraglia <jbaraglia@google.com>

File: aic_assets/models/NIC Card Mount/nic_card_mount_macro.xacro (robot description, xacro)
@@ -1,203 +1,20 @@
 <?xml version="1.0" ?>
 <robot xmlns:xacro="http://wiki.ros.org/xacro">
-  <xacro:macro name="nic_card_mount" params="prefix">
-    <!-- NIC Card Mount Link -->
-    <link name="${prefix}link">
-      <inertial>
-        <origin xyz="0 0 0" rpy="0 0 0"/>
-        <mass value="0.1"/>
-        <inertia ixx="0.001" ixy="0.0" ixz="0.0" iyy="0.001" iyz="0.0" izz="0.001"/>
-      </inertial>
-      <visual name="nic_card_mount_visual">
-        <origin xyz="0 0 0" rpy="0 0 0"/>
-        <geometry>
-          <mesh filename="package://aic_assets/models/NIC Card Mount/nic_card_mount_visual.glb"/>
-        </geometry>
-      </visual>
-      <collision name="v1015085006_collider_box">
-        <origin xyz="0.007 -0.0255 0.0775" rpy="0.0 0.0 1.570796"/>
-        <geometry>
-          <box size="0.005 0.072 0.155"/>
-        </geometry>
-      </collision>
-      <collision name="v1015085006_collider_box_001">
-        <origin xyz="-0.048467 -0.0155 0.162" rpy="0.0 0.0 1.570796"/>
-        <geometry>
-          <box size="0.025 0.039374 0.014"/>
-        </geometry>
-      </collision>
-      <collision name="v1015085006_collider_box_002">
-        <origin xyz="0.0405 -0.01425 0.1055" rpy="0.0 0.0 1.570796"/>
-        <geometry>
-          <box size="0.0275 0.005 0.103"/>
-        </geometry>
-      </collision>
-      <collision name="v1015085006_collider_box_003">
-        <origin xyz="0.0 -0.0125 0.0055" rpy="0.0 0.0 1.570796"/>
-        <geometry>
-          <box size="0.031 0.058 0.011"/>
-        </geometry>
-      </collision>
-      <collision name="v1015085006_collider_box004_collider_box">
-        <origin xyz="-0.045132 -0.0255 0.137803" rpy="0.0 0.0 1.570796"/>
-        <geometry>
-          <box size="0.005 0.036343 0.034395"/>
-        </geometry>
-      </collision>
-    </link>
-    <!-- NIC Card Link -->
-    <link name="${prefix}card_link">
-      <inertial>
-        <origin xyz="0 0 0" rpy="0 0 0"/>
-        <mass value="0.15"/>
-        <inertia ixx="0.001" ixy="0.0" ixz="0.0" iyy="0.001" iyz="0.0" izz="0.001"/>
-      </inertial>
-      <visual name="nic_card_visual">
-        <origin xyz="0 0 0" rpy="0 0 0"/>
-        <geometry>
-          <mesh filename="package://aic_assets/models/NIC Card Mount/nic_card_visual.glb"/>
-        </geometry>
-      </visual>
-      <collision name="pcb_collider_box">
-        <origin xyz="0.0 0.0 -0.0008" rpy="0.0 0.0 0.0"/>
-        <geometry>
-          <box size="0.056 0.145 0.0016"/>
-        </geometry>
-      </collision>
-      <collision name="pcb_collider_box_001">
-        <origin xyz="0.0065 -0.0025 -0.0008" rpy="0.0 0.0 0.0"/>
-        <geometry>
-          <box size="0.069 0.051 0.0016"/>
-        </geometry>
-      </collision>
-      <collision name="pcb_collider_box_002">
-        <origin xyz="0.004 -0.02475 -0.0008" rpy="0.0 0.0 0.0"/>
-        <geometry>
-          <box size="0.064 0.0955 0.0016"/>
-        </geometry>
-      </collision>
-      <collision name="cube001_collider_box">
-        <origin xyz="0.025006 -0.00041 0.00575" rpy="0.0 0.0 0.0"/>
-        <geometry>
-          <box size="0.004 0.14 0.0115"/>
-        </geometry>
-      </collision>
-      <collision name="cube001_collider_box_001">
-        <origin xyz="-0.0029 -0.0015 0.008" rpy="0.0 0.0 0.0"/>
-        <geometry>
-          <box size="0.047 0.052 0.011"/>
-        </geometry>
-      </collision>
-      <collision name="cube001_collider_box_002">
-        <origin xyz="-0.0029 -0.0015 0.001228" rpy="0.0 0.0 0.0"/>
-        <geometry>
-          <box size="0.043 0.048 0.003149"/>
-        </geometry>
-      </collision>
-      <collision name="10099100-011lfc001_collider_box">
-        <origin xyz="-0.017799 -0.052954 0.00548" rpy="3.128092 0.0 0.0"/>
-        <geometry>
-          <box size="0.001099 0.04872 0.011083"/>
-        </geometry>
-      </collision>
-      <collision name="10099100-011lfc001_collider_box.001">
-        <origin xyz="-0.002687 -0.052954 0.005461" rpy="3.128092 0.0 0.0"/>
-        <geometry>
-          <box size="0.001125 0.04872 0.011121"/>
-        </geometry>
-      </collision>
-      <collision name="10099100-011lfc001_collider_box.002">
-        <origin xyz="-0.010237 -0.052889 0.010234" rpy="3.128092 0.0 0.0"/>
-        <geometry>
-          <box size="0.016224 0.04872 0.000923"/>
-        </geometry>
-      </collision>
-      <collision name="10099100-011lfc001_collider_box.003">
-        <origin xyz="-0.010237 -0.053024 0.000296" rpy="3.128092 0.0 0.0"/>
-        <geometry>
-          <box size="0.016224 0.04872 0.001054"/>
-        </geometry>
-      </collision>
-      <collision name="10099100-011lfc001_collider_box.004">
-        <origin xyz="-0.010237 -0.028738 0.003845" rpy="3.128092 0.0 0.0"/>
-        <geometry>
-          <box size="0.016224 0.00025 0.013698"/>
-        </geometry>
-      </collision>
-      <collision name="10099100-011lfc001_collider_box.005">
-        <origin xyz="0.005401 -0.052954 0.00548" rpy="3.128092 0.0 0.0"/>
-        <geometry>
-          <box size="0.001099 0.04872 0.011083"/>
-        </geometry>
-      </collision>
-      <collision name="10099100-011lfc001_collider_box.006">
-        <origin xyz="0.020513 -0.052954 0.005461" rpy="3.128092 0.0 0.0"/>
-        <geometry>
-          <box size="0.001125 0.04872 0.011121"/>
-        </geometry>
-      </collision>
-      <collision name="10099100-011lfc001_collider_box.007">
-        <origin xyz="0.012963 -0.052889 0.010234" rpy="3.128092 0.0 0.0"/>
-        <geometry>
-          <box size="0.016224 0.04872 0.00092"/>
-        </geometry>
-      </collision>
-      <collision name="10099100-011lfc001_collider_box.008">
-        <origin xyz="0.012963 -0.053024 0.000296" rpy="3.128092 0.0 0.0"/>
-        <geometry>
-          <box size="0.016224 0.04872 0.001054"/>
-        </geometry>
-      </collision>
-      <collision name="10099100-011lfc001_collider_box.009">
-        <origin xyz="0.012963 -0.028738 0.003845" rpy="3.128092 0.0 0.0"/>
-        <geometry>
-          <box size="0.016224 0.00025 0.01369"/>
-        </geometry>
-      </collision>
-      <collision name="plane001_collider_box">
-        <origin xyz="-0.007649 -0.074646 -0.0007515" rpy="0.0 0.0 0.0"/>
-        <geometry>
-          <box size="0.113402 0.000875 0.003449"/>
-        </geometry>
-      </collision>
-      <collision name="plane001_collider_box.001">
-        <origin xyz="-0.007649 -0.074646 0.01352" rpy="0.0 0.0 0.0"/>
-        <geometry>
-          <box size="0.113402 0.000875 0.00501"/>
-        </geometry>
-      </collision>
-      <collision name="plane001_collider_box.002">
-        <origin xyz="0.038559 -0.074646 0.006455" rpy="0.0 0.0 0.0"/>
-        <geometry>
-          <box size="0.036181 0.000875 0.01112"/>
-        </geometry>
-      </collision>
-      <collision name="plane001_collider_box.003">
-        <origin xyz="-0.041261 -0.074646 0.006455" rpy="0.0 0.0 0.0"/>
-        <geometry>
-          <box size="0.046178 0.000875 0.011123"/>
-        </geometry>
-      </collision>
-    </link>
-    <!-- Joint connecting card to mount -->
-    <joint name="${prefix}card_joint" type="fixed">
-      <parent link="${prefix}link"/>
-      <child link="${prefix}card_link"/>
-      <origin xyz="0 -0.01785 0.0799" rpy="-1.57 0 0"/>
-    </joint>
-    <!-- SFP Port 0 Link -->
-    <link name="${prefix}sfp_port_0_link"/>
-    <joint name="${prefix}sfp_port_0_joint" type="fixed">
-      <parent link="${prefix}card_link"/>
-      <child link="${prefix}sfp_port_0_link"/>
-      <origin xyz="0.01295 -0.031572 0.00501" rpy="4.69895 0 0"/>
-    </joint>
-    <!-- SFP Port 1 Link -->
-    <link name="${prefix}sfp_port_1_link"/>
-    <joint name="${prefix}sfp_port_1_joint" type="fixed">
-      <parent link="${prefix}card_link"/>
-      <child link="${prefix}sfp_port_1_link"/>
-      <origin xyz="-0.01025 -0.031572 0.00501" rpy="4.69895 0 0"/>
-    </joint>
+  <xacro:macro name="nic_card_mount" params="prefix pose">
+    <gazebo>
+      <include>
+        <name>${prefix}</name>
+        <uri>package://aic_assets/models/NIC Card Mount</uri>
+        <pose>${pose}</pose>
+        <plugin
+          filename="gz-sim-touchplugin-system"
+          name="gz::sim::systems::TouchPlugin">
+          <target>sfp_module</target>
+          <time>1</time>
+          <namespace>${prefix}</namespace>
+          <enabled>true</enabled>
+        </plugin>
+      </include>
+    </gazebo>
   </xacro:macro>
 </robot>

File: aic_assets/models/SC Port/sc_port_macro.xacro (robot description, xacro)
@@ -1,78 +1,20 @@
 <?xml version="1.0" ?>
 <robot xmlns:xacro="http://wiki.ros.org/xacro">
-  <xacro:macro name="sc_port" params="prefix">
-    <link name="${prefix}link">
-      <inertial>
-        <origin xyz="0 0 0" rpy="0 0 0"/>
-        <mass value="0.04"/>
-        <inertia ixx="0.0001" ixy="0.0" ixz="0.0" iyy="0.0001" iyz="0.0" izz="0.0001"/>
-      </inertial>
-      <visual name="sc_port_visual">
-        <origin xyz="0 0 0" rpy="0 0 0"/>
-        <geometry>
-          <mesh filename="package://aic_assets/models/SC Port/sc_port_visual.glb"/>
-        </geometry>
-      </visual>
-      <collision name="cube_collider_box">
-        <origin xyz="0.011922 0.0 0.0" rpy="0.0 0.0 0.0"/>
-        <geometry>
-          <box size="0.001937 0.027432 0.0093"/>
-        </geometry>
-      </collision>
-      <collision name="cube_collider_box_001">
-        <origin xyz="0.0 0.0 0.004225" rpy="0.0 0.0 0.0"/>
-        <geometry>
-          <box size="0.025781 0.0108 0.00085"/>
-        </geometry>
-      </collision>
-      <collision name="cube_collider_box_mid">
-        <origin xyz="0.0 0.0 0.004225" rpy="0.0 0.0 0.0"/>
-        <geometry>
-          <box size="0.0103 0.027432 0.00085"/>
-        </geometry>
-      </collision>
-      <collision name="cube_collider_box_mid02">
-        <origin xyz="0.01 0.0 0.004225" rpy="0.0 0.0 0.0"/>
-        <geometry>
-          <box size="0.005 0.027432 0.00085"/>
-        </geometry>
-      </collision>
-      <collision name="cube_collider_box_mid03">
-        <origin xyz="-0.01 0.0 0.004225" rpy="0.0 0.0 0.0"/>
-        <geometry>
-          <box size="0.005 0.027432 0.00085"/>
-        </geometry>
-      </collision>
-      <collision name="cube_collider_box_002">
-        <origin xyz="0.0 0.0 -0.004225" rpy="0.0 0.0 0.0"/>
-        <geometry>
-          <box size="0.02565 0.027432 0.00085"/>
-        </geometry>
-      </collision>
-      <collision name="cube_collider_box_003">
-        <origin xyz="-0.011922 0.0 0.0" rpy="0.0 0.0 0.0"/>
-        <geometry>
-          <box size="0.001937 0.027432 0.0093"/>
-        </geometry>
-      </collision>
-      <collision name="cube_collider_box_004">
-        <origin xyz="-0.014683 0.0 0.0" rpy="0.0 0.0 0.0"/>
-        <geometry>
-          <box size="0.005484 0.003048 0.0093"/>
-        </geometry>
-      </collision>
-      <collision name="cube_collider_box_005">
-        <origin xyz="0.014683 0.0 0.0" rpy="0.0 0.0 0.0"/>
-        <geometry>
-          <box size="0.005484 0.003048 0.0093"/>
-        </geometry>
-      </collision>
-      <collision name="cube_collider_box_006">
-        <origin xyz="0.0 0.0 0.0" rpy="0.0 0.0 0.0"/>
-        <geometry>
-          <box size="0.003492 0.027432 0.0093"/>
-        </geometry>
-      </collision>
-    </link>
+  <xacro:macro name="sc_port" params="prefix pose">
+    <gazebo>
+      <include>
+        <name>${prefix}</name>
+        <uri>package://aic_assets/models/SC Port</uri>
+        <pose>${pose}</pose>
+        <plugin
+          filename="gz-sim-touchplugin-system"
+          name="gz::sim::systems::TouchPlugin">
+          <target>sc_plug</target>
+          <time>1</time>
+          <namespace>${prefix}</namespace>
+          <enabled>true</enabled>
+        </plugin>
+      </include>
+    </gazebo>
   </xacro:macro>
 </robot>

File: aic_description/urdf/cable.sdf.xacro (robot description, xacro)
@@ -9,4 +9,6 @@
       <plugin filename="CablePlugin" name="aic_gazebo::CablePlugin">
         <cable_connection_0_link>lc_plug_link</cable_connection_0_link>
+        <!-- this should match the target port's <namespace> parameter in its xacro file -->
+        <cable_connection_0_port>nic_card_mount_0</cable_connection_0_port>
         <cable_connection_1_link>sc_plug_link</cable_connection_1_link>
         <end_effector_model>ur5e</end_effector_model>

File: aic_description/urdf/task_board.urdf.xacro (robot description, xacro)
@@ -156,64 +156,71 @@
   <!-- SC Port 0 -->
   <xacro:if value="$(arg sc_port_0_present)">
-    <xacro:sc_port prefix="sc_port_0_"/>
-    <joint name="sc_port_0_joint" type="fixed">
-      <parent link="task_board_base_link"/>
-      <child link="sc_port_0_link"/>
-      <origin xyz="${-0.075 + $(arg sc_port_0_translation)} 0.0295 0.0145" rpy="${1.57 + $(arg sc_port_0_roll)} $(arg sc_port_0_pitch) ${1.57 + $(arg sc_port_0_yaw)}"/>
-    </joint>
+    <xacro:sc_port prefix="sc_port_0" pose="${-0.075 + $(arg sc_port_0_translation)} 0.0295 0.0145 ${1.57 + $(arg sc_port_0_roll)} $(arg sc_port_0_pitch) ${1.57 + $(arg sc_port_0_yaw)}"/>
+    <gazebo>
+      <joint name="sc_port_0_joint" type="fixed">
+        <parent>task_board_base_link</parent>
+        <child>sc_port_0::sc_port_link</child>
+      </joint>
+    </gazebo>
   </xacro:if>
   <!-- SC Port 1 -->
   <xacro:if value="$(arg sc_port_1_present)">
-    <xacro:sc_port prefix="sc_port_1_"/>
-    <joint name="sc_port_1_joint" type="fixed">
-      <parent link="task_board_base_link"/>
-      <child link="sc_port_1_link"/>
-      <origin xyz="${-0.075 + $(arg sc_port_1_translation)} 0.0705 0.0145" rpy="${1.57 + $(arg sc_port_1_roll)} $(arg sc_port_1_pitch) ${1.57 + $(arg sc_port_1_yaw)}"/>
-    </joint>
+    <xacro:sc_port prefix="sc_port_1" pose="${-0.075 + $(arg sc_port_1_translation)} 0.0705 0.0145 ${1.57 + $(arg sc_port_1_roll)} $(arg sc_port_1_pitch) ${1.57 + $(arg sc_port_1_yaw)}"/>
+    <gazebo>
+      <joint name="sc_port_1_joint" type="fixed">
+        <parent>task_board_base_link</parent>
+        <child>sc_port_1::sc_port_link</child>
+      </joint>
+    </gazebo>
   </xacro:if>
   <!-- NIC Card Mount 0 (left-most) -->
   <xacro:if value="$(arg nic_card_mount_0_present)">
-    <xacro:nic_card_mount prefix="nic_card_mount_0_"/>
-    <joint name="nic_card_mount_0_joint" type="fixed">
-      <parent link="task_board_base_link"/>
-      <child link="nic_card_mount_0_link"/>
-      <origin xyz="${-0.081418 + $(arg nic_card_mount_0_translation)} -0.1745 0.01" rpy="$(arg nic_card_mount_0_roll) $(arg nic_card_mount_0_pitch) $(arg nic_card_mount_0_yaw)"/>
-    </joint>
+    <xacro:nic_card_mount prefix="nic_card_mount_0" pose="${-0.081418 + $(arg nic_card_mount_0_translation)} -0.1745 0.01 $(arg nic_card_mount_0_roll) $(arg nic_card_mount_0_pitch) $(arg nic_card_mount_0_yaw)"/>
+    <gazebo>
+      <joint name="nic_card_mount_0_joint" type="fixed">
+        <parent>task_board_base_link</parent>
+        <child>nic_card_mount_0::nic_card_mount_link</child>
+      </joint>
+    </gazebo>
   </xacro:if>
   <!-- NIC Card Mount 1 -->
   <xacro:if value="$(arg nic_card_mount_1_present)">
-    <xacro:nic_card_mount prefix="nic_card_mount_1_"/>
-    <joint name="nic_card_mount_1_joint" type="fixed">
-      <parent link="task_board_base_link"/>
-      <child link="nic_card_mount_1_link"/>
-      <origin xyz="${-0.081418 + $(arg nic_card_mount_1_translation)} -0.1345 0.01" rpy="$(arg nic_card_mount_1_roll) $(arg nic_card_mount_1_pitch) $(arg nic_card_mount_1_yaw)"/>
-    </joint>
+    <xacro:nic_card_mount prefix="nic_card_mount_1" pose="${-0.081418 + $(arg nic_card_mount_1_translation)} -0.1345 0.01 $(arg nic_card_mount_1_roll) $(arg nic_card_mount_1_pitch) $(arg nic_card_mount_1_yaw)"/>
+    <gazebo>
+      <joint name="nic_card_mount_1_joint" type="fixed">
+        <parent>task_board_base_link</parent>
+        <child>nic_card_mount_1::nic_card_mount_link</child>
+      </joint>
+    </gazebo>
   </xacro:if>
   <!-- NIC Card Mount 2 (center) -->
   <xacro:if value="$(arg nic_card_mount_2_present)">
-    <xacro:nic_card_mount prefix="nic_card_mount_2_"/>
-    <joint name="nic_card_mount_2_joint" type="fixed">
-      <parent link="task_board_base_link"/>
-      <child link="nic_card_mount_2_link"/>
-      <origin xyz="${-0.081418 + $(arg nic_card_mount_2_translation)} -0.0945 0.01" rpy="$(arg nic_card_mount_2_roll) $(arg nic_card_mount_2_pitch) $(arg nic_card_mount_2_yaw)"/>
-    </joint>
+    <xacro:nic_card_mount prefix="nic_card_mount_2" pose="${-0.081418 + $(arg nic_card_mount_2_translation)} -0.0945 0.01" rpy="$(arg nic_card_mount_2_roll) $(arg nic_card_mount_2_pitch) $(arg nic_card_mount_2_yaw)"/>
+    <gazebo>
+      <joint name="nic_card_mount_2_joint" type="fixed">
+        <parent>task_board_base_link</parent>
+        <child>nic_card_mount_2::nic_card_mount_link</child>
+      </joint>
+    </gazebo>
   </xacro:if>
   <!-- NIC Card Mount 3 -->
   <xacro:if value="$(arg nic_card_mount_3_present)">
-    <xacro:nic_card_mount prefix="nic_card_mount_3_"/>
-    <joint name="nic_card_mount_3_joint" type="fixed">
-      <parent link="task_board_base_link"/>
-      <child link="nic_card_mount_3_link"/>
-      <origin xyz="${-0.081418 + $(arg nic_card_mount_3_translation)} -0.0545 0.01" rpy="$(arg nic_card_mount_3_roll) $(arg nic_card_mount_3_pitch) $(arg nic_card_mount_3_yaw)"/>
-    </joint>
+    <xacro:nic_card_mount prefix="nic_card_mount_3 ${-0.081418 + $(arg nic_card_mount_3_translation)} -0.0545 0.01" rpy="$(arg nic_card_mount_3_roll) $(arg nic_card_mount_3_pitch) $(arg nic_card_mount_3_yaw)"/>
+    <gazebo>
+      <joint name="nic_card_mount_3_joint" type="fixed">
+        <parent>task_board_base_link</parent>
+        <child>nic_card_mount_3::nic_card_mount_link</child>
+      </joint>
+    </gazebo>
   </xacro:if>
   <!-- NIC Card Mount 4 (right-most) -->
   <xacro:if value="$(arg nic_card_mount_4_present)">
-    <xacro:nic_card_mount prefix="nic_card_mount_4_"/>
-    <joint name="nic_card_mount_4_joint" type="fixed">
-      <parent link="task_board_base_link"/>
-      <child link="nic_card_mount_4_link"/>
-      <origin xyz="${-0.081418 + $(arg nic_card_mount_4_translation)} -0.0145 0.01" rpy="$(arg nic_card_mount_4_roll) $(arg nic_card_mount_4_pitch) $(arg nic_card_mount_4_yaw)"/>
-    </joint>
+    <xacro:nic_card_mount prefix="nic_card_mount_4" pose="${-0.081418 + $(arg nic_card_mount_4_translation)} -0.0145 0.01 $(arg nic_card_mount_4_roll) $(arg nic_card_mount_4_pitch) $(arg nic_card_mount_4_yaw)"/>
+    <gazebo>
+      <joint name="nic_card_mount_4_joint" type="fixed">
+        <parent>task_board_base_link</parent>
+        <child>nic_card_mount_4::nic_card_mount_link</child>
+      </joint>
+    </gazebo>
   </xacro:if>
   <gazebo>
