Commit message: update basler camera xacro

File: aic_assets/models/Basler Camera/basler_camera_macro.xacro (robot description, xacro)
@@ -2,10 +2,7 @@
 <robot xmlns:xacro="http://wiki.ros.org/xacro">
   <xacro:macro name="basler_camera" params="name tf_prefix use_sim_cam">
-    <xacro:property name="x_rot" value="1.5708"/>
-    <xacro:property name="y_rot" value="0.0"/>
-    <xacro:property name="z_rot" value="1.5708"/>
     <link name="${tf_prefix}basler_cam_link">
       <inertial>
-        <origin xyz="0 0 0" rpy="${x_rot} ${y_rot} ${z_rot}"/>
+        <origin xyz="0 0 0" rpy="0 0 0"/>
         <mass value="0.1"/>
         <inertia ixx="0.00002083" ixy="0" ixz="0"
@@ -14,26 +11,25 @@
       </inertial>
       <visual name="basler_cam_visual">
-        <origin xyz="0 0 0" rpy="${x_rot} ${y_rot} ${z_rot}"/>
         <geometry>
           <mesh filename="package://aic_assets/models/Basler Camera/basler_cam_visual.glb"/>
         </geometry>
       </visual>
-      <collision name="lens001_collider_cylinder">
-        <origin xyz="0.013336 0 0" rpy="${x_rot} ${y_rot} ${z_rot}"/>
+      <collision name="135368670234ip01880201_collider_box">
+        <origin xyz="-0.0 -0.0144 0.00255" rpy="3.141593 -0.0 0.0"/>
         <geometry>
-          <cylinder radius="0.016429" length="0.040108"/>
+          <box size="0.029 0.029 0.0483"/>
         </geometry>
       </collision>
-      <collision name="basler_ace2_gige027_collider_box">
-        <origin xyz="-0.031178 0 0" rpy="0 0 0"/>
+      <collision name="sphere_collider_cylinder">
+        <origin xyz="0.0 -0.014507 0.04833" rpy="0 0 0"/>
         <geometry>
-          <box size="0.04919 0.029 0.029"/>
+          <cylinder radius="0.015631" length="0.04326"/>
         </geometry>
       </collision>
       <!-- the IO connector on the back of the camera -->
-      <collision name="basler_ace2_gige011_collider_cylinder">
-        <origin xyz="-0.058082 -0.005773 -0.0081" rpy="0 1.5708 0"/>
+      <collision name="59871rev000001_collider_box">
+        <origin xyz="-0.008138 -0.000452 0.052687" rpy="-1.587325 0.0 -2.633954"/>
         <geometry>
-          <cylinder radius="0.005145" length="0.008255"/>
+          <box size="0.003998 0.011586 0.006875"/>
         </geometry>
       </collision>

Commit message: Update camera, sensor, and optical frames

File: aic_assets/models/Basler Camera/basler_camera_macro.xacro (robot description, xacro)
@@ -2,5 +2,5 @@
 <robot xmlns:xacro="http://wiki.ros.org/xacro">
   <xacro:macro name="basler_camera" params="name tf_prefix use_sim_cam">
-    <link name="${tf_prefix}basler_cam_link">
+    <link name="${tf_prefix}camera_link">
       <inertial>
         <origin xyz="0 0 0" rpy="0 0 0"/>
@@ -11,28 +11,42 @@
       </inertial>
       <visual name="basler_cam_visual">
+        <origin xyz="0 0 0" rpy="-1.5708 0 -1.5708"/>
         <geometry>
           <mesh filename="package://aic_assets/models/Basler Camera/basler_cam_visual.glb"/>
         </geometry>
       </visual>
-      <collision name="135368670234ip01880201_collider_box">
-        <origin xyz="-0.0 -0.0144 0.00255" rpy="3.141593 -0.0 0.0"/>
+      <collision name="body_collider_box">
+        <origin xyz="0.00255 0 0.0145" rpy="0 0 0"/>
         <geometry>
-          <box size="0.029 0.029 0.0483"/>
+          <box size="0.0483 0.029 0.029"/>
         </geometry>
       </collision>
-      <collision name="sphere_collider_cylinder">
-        <origin xyz="0.0 -0.014507 0.04833" rpy="0 0 0"/>
+      <collision name="lens_collider_cylinder">
+        <origin xyz="0.04833 0 0.0145" rpy="0 1.5708 0"/>
         <geometry>
           <cylinder radius="0.015631" length="0.04326"/>
         </geometry>
       </collision>
-      <!-- the IO connector on the back of the camera -->
-      <collision name="59871rev000001_collider_box">
-        <origin xyz="-0.008138 -0.000452 0.052687" rpy="-1.587325 0.0 -2.633954"/>
-        <geometry>
-          <box size="0.003998 0.011586 0.006875"/>
-        </geometry>
-      </collision>
     </link>
+    <link name="${tf_prefix}sensor_link">
+      <!-- inertial property required for valid conversion to SDF,
+        so we set a tiny mass and M.O.I. here -->
+      <inertial>
+        <origin xyz="0 0 0" rpy="0 0 0"/>
+        <mass value="0.001"/>
+        <inertia ixx="0.000001" ixy="0" ixz="0"
+                 iyy="0.000001" iyz="0"
+                 izz="0.000001"/>
+      </inertial>
+    </link>
+    <!-- The sensor surface is 21.174mm in front of the M3 mounting hole -->
+    <joint name="${tf_prefix}attach_sensor_link" type="fixed">
+      <origin xyz="0.02174 0 0.0145" rpy="0 0 0"/>
+      <parent link="${tf_prefix}camera_link"/>
+      <child link="${tf_prefix}sensor_link"/>
+    </joint>
+    <gazebo reference="${tf_prefix}attach_sensor_link">
+      <preserveFixedJoint>true</preserveFixedJoint>
+    </gazebo>
     <link name="${tf_prefix}optical">
       <!-- inertial property required for valid conversion to SDF,
@@ -46,33 +60,12 @@
       </inertial>
     </link>
+    <!-- The optical frame is at the same origin as the sensor frame
+         but is Z=forward, rather than Z=up. -->
     <joint name="${tf_prefix}attach_optical" type="fixed">
       <origin xyz="0 0 0" rpy="-1.5708 0 -1.5708"/>
-      <parent link="${tf_prefix}basler_cam_link"/>
+      <parent link="${tf_prefix}sensor_link"/>
       <child link="${tf_prefix}optical"/>
     </joint>
     <gazebo reference="${tf_prefix}attach_optical">
-      <preserveFixedJoint>true</preserveFixedJoint>
-    </gazebo>
-    <link name="${tf_prefix}sensor_link">
-      <!-- inertial property required for valid conversion to SDF,
-        so we set a tiny mass and M.O.I. here -->
-      <inertial>
-        <origin xyz="0 0 0" rpy="0 0 0"/>
-        <mass value="0.001"/>
-        <inertia ixx="0.000001" ixy="0" ixz="0"
-                 iyy="0.000001" iyz="0"
-                 izz="0.000001"/>
-      </inertial>
-    </link>
-    <!-- Currently the sensor_link is the same location as the
-         cam_link frame. However, we may adjust this in the future
-         if the lens focal point ends up being somewhat forward or
-         backward of the current estimate. -->
-    <joint name="${tf_prefix}attach_sensor_link" type="fixed">
-      <origin xyz="0 0 0" rpy="0 0 0"/>
-      <parent link="${tf_prefix}basler_cam_link"/>
-      <child link="${tf_prefix}sensor_link"/>
-    </joint>
-    <gazebo reference="${tf_prefix}attach_sensor_link">
       <preserveFixedJoint>true</preserveFixedJoint>
     </gazebo>

File: aic_description/urdf/ur_gz.urdf.xacro (robot description, xacro)
@@ -157,7 +157,7 @@
   </joint>
   <joint name="attach_wrist_camera_1" type="fixed">
-    <origin xyz="0 -0.1077 -.00719" rpy="-0.261799 0 0"/>
-    <parent link="$(arg cam_mount_tf_prefix)cam_mount_link"/>
-    <child link="$(arg wrist_camera_1_tf_prefix)basler_cam_link"/>
+    <origin xyz="0 -0.1077 -.00719" rpy="0 -1.30899630 1.57079623"/>
+    <parent link="$(arg cam_mount_tf_prefix)cam_mount_link"/>
+    <child link="$(arg wrist_camera_1_tf_prefix)camera_link"/>
   </joint>
   <!-- ********************
@@ -165,7 +165,7 @@
        ******************** -->
   <joint name="attach_wrist_camera_2" type="fixed">
-    <origin xyz="-0.09326 -0.053843 -0.007188" rpy="-0.261799 0.0 -1.047198"/>
-    <parent link="$(arg cam_mount_tf_prefix)cam_mount_link"/>
-    <child link="$(arg wrist_camera_2_tf_prefix)basler_cam_link"/>
+    <origin xyz="-0.09326 -0.053843 -0.007188" rpy="0 -1.30899630 0.523599027"/>
+    <parent link="$(arg cam_mount_tf_prefix)cam_mount_link"/>
+    <child link="$(arg wrist_camera_2_tf_prefix)camera_link"/>
   </joint>
   <!-- ********************
@@ -173,7 +173,7 @@
        ******************** -->
   <joint name="attach_wrist_camera_3" type="fixed">
-    <origin xyz="0.09326 -0.053843 -0.007188" rpy="-0.261799 0.0 1.047198"/>
-    <parent link="$(arg cam_mount_tf_prefix)cam_mount_link"/>
-    <child link="$(arg wrist_camera_3_tf_prefix)basler_cam_link"/>
+    <origin xyz="0.09326 -0.053843 -0.007188" rpy="0 -1.30899630 2.61799343"/>
+    <parent link="$(arg cam_mount_tf_prefix)cam_mount_link"/>
+    <child link="$(arg wrist_camera_3_tf_prefix)camera_link"/>
   </joint>
   <joint name="attach_gripper" type="fixed">

Commit message: set masses to small values for links no in the kinematic chain and remove repeated <inertial> blocks (#84)

File: aic_assets/models/Basler Camera/basler_camera_macro.xacro (robot description, xacro)
@@ -5,5 +5,5 @@
       <inertial>
         <origin xyz="0 0 0" rpy="0 0 0"/>
-        <mass value="0.1"/>
+        <mass value="0.001"/>
         <inertia ixx="0.00002083" ixy="0" ixz="0"
                  iyy="0.00002083" iyz="0"

File: aic_assets/models/Robotiq Hand-E/robotiq_hande_macro.xacro (robot description, xacro)
@@ -43,5 +43,5 @@
       <inertial>
         <origin xyz="0 0 0" rpy="0 0 0"/>
-        <mass value="0.2"/>
+        <mass value="0.001"/>
         <inertia ixx="0.0001" ixy="0" ixz="0"
                  iyy="0.00009" iyz="0"
@@ -78,14 +78,9 @@
         </geometry>
       </collision>
-      <inertial>
-        <origin xyz="0 0 0" rpy="0 0 0"/>
-        <mass value="0.2"/>
-        <inertia ixx="0.0001" ixy="0.0" ixz="0.0" iyy="0.00009" iyz="0.0" izz="0.00003"/>
-      </inertial>
     </link>
     <link name="${tf_prefix}hande_finger_link_r">
       <inertial>
         <origin xyz="0 0 0" rpy="0 0 0"/>
-        <mass value="0.2"/>
+        <mass value="0.001"/>
         <inertia ixx="0.0001" ixy="0" ixz="0"
                  iyy="0.00009" iyz="0"
@@ -122,9 +117,4 @@
         </geometry>
       </collision>
-      <inertial>
-        <origin xyz="0 0 0" rpy="0 0 0"/>
-        <mass value="0.2"/>
-        <inertia ixx="0.0001" ixy="0.0" ixz="0.0" iyy="0.00009" iyz="0.0" izz="0.00003"/>
-      </inertial>
     </link>
     <joint name="${tf_prefix}left_finger_joint" type="prismatic">
