Commit message: Update taskboard (#166)
* added v2 taskboard models

* updated necessary xacro files

* fixed nic card offset

* Update comment

Signed-off-by: Yadunund <yadunund@intrinsic.ai>

* adjusted nic card limits

* Tweak sc_rail min

Signed-off-by: Yadunund <yadunund@intrinsic.ai>

---------

Signed-off-by: Yadunund <yadunund@intrinsic.ai>
Co-authored-by: Yadunund <yadunund@intrinsic.ai>

File: aic_assets/models/LC Mount/lc_mount_macro.xacro (robot description, xacro)
@@ -15,43 +15,49 @@
       </visual>
       <collision name="v1015081011_collider_box">
-        <origin xyz="0.019353 0.0 0.0025" rpy="0.0 0.0 0.0"/>
+        <origin xyz="0.039468 0.0 0.0025" rpy="0.0 0.0 0.0"/>
         <geometry>
-          <box size="0.019294 0.01475 0.005"/>
+          <box size="0.017033 0.006 0.005"/>
         </geometry>
       </collision>
-      <collision name="v1015081011_collider_box_001">
-        <origin xyz="-0.00294 0.0 0.0025" rpy="0.0 0.0 0.0"/>
+      <collision name="v1015081011_collider_box.001">
+        <origin xyz="0.006285 0.0 0.0025" rpy="0.0 0.0 0.0"/>
         <geometry>
-          <box size="0.01212 0.01475 0.005"/>
+          <box size="0.018569 0.006 0.005"/>
         </geometry>
       </collision>
-      <collision name="v1015081011_collider_box_002">
-        <origin xyz="0.004062 0.0 0.014555" rpy="0.0 -0.785398 0.0"/>
+      <collision name="v1015081011_collider_box.002">
+        <origin xyz="0.016889 0.0 0.014186" rpy="0.0 -0.785398 0.0"/>
         <geometry>
-          <box size="0.014258 0.01475 0.002"/>
+          <box size="0.014269 0.01475 0.003054"/>
         </geometry>
       </collision>
-      <collision name="v1015081011_collider_box_003">
-        <origin xyz="0.015992 0.0 0.004149" rpy="0.0 -0.785398 0.0"/>
+      <collision name="v1015081011_collider_box.003">
+        <origin xyz="0.029227 0.0 0.003364" rpy="0.0 -0.785398 0.0"/>
         <geometry>
-          <box size="0.012103 0.01475 0.010218"/>
+          <box size="0.012103 0.01475 0.007998"/>
         </geometry>
       </collision>
-      <collision name="v1015081011_collider_box_004">
-        <origin xyz="0.001043 0.0 0.003076" rpy="0.0 -0.785398 0.0"/>
+      <collision name="v1015081011_collider_box.004">
+        <origin xyz="0.013496 0.0 0.003079" rpy="0.0 -0.785398 0.0"/>
         <geometry>
-          <box size="0.006246 0.01475 0.013841"/>
+          <box size="0.006255 0.01475 0.013841"/>
         </geometry>
       </collision>
-      <collision name="v1015081011_collider_box_005">
-        <origin xyz="0.00925 0.006437 0.009368" rpy="0.0 -0.785398 0.0"/>
+      <collision name="v1015081011_collider_box.005">
+        <origin xyz="0.022239 0.00575 0.008836" rpy="0.0 -0.785398 0.0"/>
         <geometry>
-          <box size="0.014258 0.001875 0.014086"/>
+          <box size="0.014269 0.00325 0.015602"/>
         </geometry>
       </collision>
-      <collision name="v1015081011_collider_box_006">
-        <origin xyz="0.009324 -0.006438 0.009293" rpy="0.0 -0.785398 0.0"/>
+      <collision name="v1015081011_collider_box.006">
+        <origin xyz="0.02227 -0.004513 0.008805" rpy="0.0 -0.785398 0.0"/>
         <geometry>
-          <box size="0.014258 0.001875 0.013874"/>
+          <box size="0.014269 0.005725 0.015265"/>
+        </geometry>
+      </collision>
+      <collision name="v1015081011_collider_box.007">
+        <origin xyz="0.032739 0.0 0.010179" rpy="0.0 -0.785398 0.0"/>
+        <geometry>
+          <box size="0.009041 0.0065 0.001804"/>
         </geometry>
       </collision>

File: aic_assets/models/SC Mount/sc_mount_macro.xacro (robot description, xacro)
@@ -15,17 +15,17 @@
       </visual>
       <collision name="v1015079011_collider_box">
-        <origin xyz="0.035449 0.0 0.0025" rpy="0.0 0.0 0.0"/>
+        <origin xyz="0.039002 0.0 0.0025" rpy="0.0 0.0 0.0"/>
         <geometry>
-          <box size="0.015101 0.014 0.005"/>
+          <box size="0.017747 0.014 0.005"/>
         </geometry>
       </collision>
-      <collision name="v1015079011_collider_box_001">
-        <origin xyz="0.020068 -0.0054 0.013451" rpy="0.0 0.785398 0.0"/>
+      <collision name="v1015079011_collider_box.001">
+        <origin xyz="0.022568 -0.0054 0.013451" rpy="0.0 0.785398 0.0"/>
         <geometry>
           <box size="0.025812 0.0032 0.013799"/>
         </geometry>
       </collision>
-      <collision name="v1015079011_collider_box_002">
-        <origin xyz="0.020068 0.00585 0.013451" rpy="0.0 0.785398 0.0"/>
+      <collision name="v1015079011_collider_box.002">
+        <origin xyz="0.022568 0.00585 0.013451" rpy="0.0 0.785398 0.0"/>
         <geometry>
           <box size="0.025812 0.0023 0.013799"/>
@@ -33,29 +33,29 @@
       </collision>
       <collision name="v1015079011_collider_box003_collider_box">
-        <origin xyz="0.01165 0.0 0.02187" rpy="0.0 0.785398 0.0"/>
+        <origin xyz="0.01415 0.0 0.02187" rpy="0.0 0.785398 0.0"/>
         <geometry>
           <box size="0.002 0.014 0.013799"/>
         </geometry>
       </collision>
-      <collision name="v1015079011_collider_box003_collider_box_001">
-        <origin xyz="0.028564 0.0 0.004956" rpy="0.0 0.785398 0.0"/>
+      <collision name="v1015079011_collider_box003_collider_box.001">
+        <origin xyz="0.031064 0.0 0.004956" rpy="0.0 0.785398 0.0"/>
         <geometry>
           <box size="0.001842 0.014 0.013799"/>
         </geometry>
       </collision>
-      <collision name="v1015079011_collider_box003_collider_box_002">
-        <origin xyz="0.008208 0.0 0.0025" rpy="0.0 0.0 0.0"/>
+      <collision name="v1015079011_collider_box003_collider_box.002">
+        <origin xyz="0.009506 0.0 0.0025" rpy="0.0 0.0 0.0"/>
         <geometry>
-          <box size="0.02236 0.014 0.005"/>
+          <box size="0.024957 0.014 0.005"/>
         </geometry>
       </collision>
-      <collision name="v1015079011_collider_box003_collider_box_003">
-        <origin xyz="0.015274 0.0 0.008656" rpy="0.0 0.785398 0.0"/>
+      <collision name="v1015079011_collider_box003_collider_box.003">
+        <origin xyz="0.017774 0.0 0.008656" rpy="0.0 0.785398 0.0"/>
         <geometry>
           <box size="0.025812 0.014 0.001239"/>
         </geometry>
       </collision>
-      <collision name="v1015079011_collider_box003_collider_box_004">
-        <origin xyz="0.032889 0.0 0.004624" rpy="0.0 0.0 0.0"/>
+      <collision name="v1015079011_collider_box003_collider_box.004">
+        <origin xyz="0.035389 0.0 0.004624" rpy="0.0 0.0 0.0"/>
         <geometry>
           <box size="0.002221 0.014 0.009249"/>
@@ -63,5 +63,5 @@
       </collision>
       <collision name="v1015079011_collider_box003_collider_box004_collider_box">
-        <origin xyz="0.007045 0.0 0.008711" rpy="0.0 0.0 0.0"/>
+        <origin xyz="0.009545 0.0 0.008711" rpy="0.0 0.0 0.0"/>
         <geometry>
           <box size="0.00209 0.014 0.017422"/>

File: aic_assets/models/Task Board Base/task_board_base_macro.xacro (robot description, xacro)
@@ -17,5 +17,5 @@
         <origin xyz="0.0 -0.10 0.0075" rpy="0.0 0.0 0.0"/>
         <geometry>
-          <box size="0.3 0.228 0.005"/>
+          <box size="0.3 0.228 0.009"/>
         </geometry>
       </collision>
@@ -23,5 +23,5 @@
         <origin xyz="0.0 0.149 0.0075" rpy="0.0 0.0 0.0"/>
         <geometry>
-          <box size="0.3 0.127 0.005"/>
+          <box size="0.3 0.127 0.009"/>
         </geometry>
       </collision>
@@ -30,5 +30,5 @@
         <origin xyz="-0.075 0.05 0.0075" rpy="0.0 0.0 0.0"/>
         <geometry>
-          <box size="0.14 0.012 0.005"/>
+          <box size="0.14 0.012 0.009"/>
         </geometry>
       </collision>
@@ -36,5 +36,5 @@
         <origin xyz="0.068 0.0 0.0075" rpy="0.0 0.0 0.0"/>
         <geometry>
-          <box size="0.165 0.425 0.005"/>
+          <box size="0.165 0.425 0.009"/>
         </geometry>
       </collision>
@@ -42,5 +42,5 @@
         <origin xyz="-0.143 0.0 0.0075" rpy="0.0 0.0 0.0"/>
         <geometry>
-          <box size="0.015 0.425 0.005"/>
+          <box size="0.015 0.425 0.009"/>
         </geometry>
       </collision>

File: aic_description/urdf/task_board.urdf.xacro (robot description, xacro)
@@ -100,5 +100,5 @@
   <!-- Instantiate Task Board Base -->
   <xacro:task_board_base prefix="task_board_"/>
-  <!-- LC Mount Rail 0: X=0.0275, Y=-0.10625 (left side, mount rail) -->
+  <!-- LC Mount Rail 0: X=0.01, Y=-0.10625 (left side, mount rail) -->
   <xacro:if value="$(arg lc_mount_rail_0_present)">
     <xacro:lc_mount prefix="lc_mount_rail_0_"/>
@@ -106,8 +106,8 @@
       <parent link="task_board_base_link"/>
       <child link="lc_mount_rail_0_link"/>
-      <origin xyz="0.0275 ${-0.10625 + $(arg lc_mount_rail_0_translation)} 0.01" rpy="$(arg lc_mount_rail_0_roll) $(arg lc_mount_rail_0_pitch) $(arg lc_mount_rail_0_yaw)"/>
-    </joint>
-  </xacro:if>
-  <!-- SFP Mount Rail 0: X=0.0535, Y=-0.10625 (left side, mount rail) -->
+      <origin xyz="0.01 ${-0.10625 + $(arg lc_mount_rail_0_translation)} 0.012" rpy="$(arg lc_mount_rail_0_roll) $(arg lc_mount_rail_0_pitch) $(arg lc_mount_rail_0_yaw)"/>
+    </joint>
+  </xacro:if>
+  <!-- SFP Mount Rail 0: X=0.055, Y=-0.10625 (left side, mount rail) -->
   <xacro:if value="$(arg sfp_mount_rail_0_present)">
     <xacro:sfp_mount prefix="sfp_mount_rail_0_"/>
@@ -115,8 +115,8 @@
       <parent link="task_board_base_link"/>
       <child link="sfp_mount_rail_0_link"/>
-      <origin xyz="0.0535 ${-0.10625 + $(arg sfp_mount_rail_0_translation)} 0.01" rpy="$(arg sfp_mount_rail_0_roll) $(arg sfp_mount_rail_0_pitch) $(arg sfp_mount_rail_0_yaw)"/>
-    </joint>
-  </xacro:if>
-  <!-- SC Mount Rail 0: X=0.0985, Y=-0.10625 (left side, mount rail) -->
+      <origin xyz="0.055 ${-0.10625 + $(arg sfp_mount_rail_0_translation)} 0.01" rpy="$(arg sfp_mount_rail_0_roll) $(arg sfp_mount_rail_0_pitch) $(arg sfp_mount_rail_0_yaw)"/>
+    </joint>
+  </xacro:if>
+  <!-- SC Mount Rail 0: X=0.1, Y=-0.10625 (left side, mount rail) -->
   <xacro:if value="$(arg sc_mount_rail_0_present)">
     <xacro:sc_mount prefix="sc_mount_rail_0_"/>
@@ -124,8 +124,8 @@
       <parent link="task_board_base_link"/>
       <child link="sc_mount_rail_0_link"/>
-      <origin xyz="0.0985 ${-0.10625 + $(arg sc_mount_rail_0_translation)} 0.01" rpy="$(arg sc_mount_rail_0_roll) $(arg sc_mount_rail_0_pitch) $(arg sc_mount_rail_0_yaw)"/>
-    </joint>
-  </xacro:if>
-  <!-- LC Mount Rail 1: X=0.0275, Y=0.10625 (right side, mount rail) -->
+      <origin xyz="0.1 ${-0.10625 + $(arg sc_mount_rail_0_translation)} 0.012" rpy="$(arg sc_mount_rail_0_roll) $(arg sc_mount_rail_0_pitch) $(arg sc_mount_rail_0_yaw)"/>
+    </joint>
+  </xacro:if>
+  <!-- LC Mount Rail 1: X=0.01, Y=0.10625 (right side, mount rail) -->
   <xacro:if value="$(arg lc_mount_rail_1_present)">
     <xacro:lc_mount prefix="lc_mount_rail_1_"/>
@@ -133,8 +133,8 @@
       <parent link="task_board_base_link"/>
       <child link="lc_mount_rail_1_link"/>
-      <origin xyz="0.0275 ${0.10625 + $(arg lc_mount_rail_1_translation)} 0.01" rpy="$(arg lc_mount_rail_1_roll) $(arg lc_mount_rail_1_pitch) $(arg lc_mount_rail_1_yaw)"/>
-    </joint>
-  </xacro:if>
-  <!-- SFP Mount Rail 1: X=0.0535, Y=0.10625 (right side, mount rail) -->
+      <origin xyz="0.01 ${0.10625 + $(arg lc_mount_rail_1_translation)} 0.012" rpy="$(arg lc_mount_rail_1_roll) $(arg lc_mount_rail_1_pitch) $(arg lc_mount_rail_1_yaw)"/>
+    </joint>
+  </xacro:if>
+  <!-- SFP Mount Rail 1: X=0.055, Y=0.10625 (right side, mount rail) -->
   <xacro:if value="$(arg sfp_mount_rail_1_present)">
     <xacro:sfp_mount prefix="sfp_mount_rail_1_"/>
@@ -142,5 +142,5 @@
       <parent link="task_board_base_link"/>
       <child link="sfp_mount_rail_1_link"/>
-      <origin xyz="0.0535 ${0.10625 + $(arg sfp_mount_rail_1_translation)} 0.01" rpy="$(arg sfp_mount_rail_1_roll) $(arg sfp_mount_rail_1_pitch) $(arg sfp_mount_rail_1_yaw)"/>
+      <origin xyz="0.055 ${0.10625 + $(arg sfp_mount_rail_1_translation)} 0.01" rpy="$(arg sfp_mount_rail_1_roll) $(arg sfp_mount_rail_1_pitch) $(arg sfp_mount_rail_1_yaw)"/>
     </joint>
   </xacro:if>
@@ -156,5 +156,5 @@
   <!-- SC Port 0 -->
   <xacro:if value="$(arg sc_port_0_present)">
-    <xacro:sc_port prefix="sc_port_0" pose="${-0.075 + $(arg sc_port_0_translation)} 0.0295 0.0145 ${1.57 + $(arg sc_port_0_roll)} $(arg sc_port_0_pitch) ${1.57 + $(arg sc_port_0_yaw)}"/>
+    <xacro:sc_port prefix="sc_port_0" pose="${-0.075 + $(arg sc_port_0_translation)} 0.0295 0.0165 ${1.57 + $(arg sc_port_0_roll)} $(arg sc_port_0_pitch) ${1.57 + $(arg sc_port_0_yaw)}"/>
     <gazebo>
       <joint name="sc_port_0_joint" type="fixed">
@@ -166,5 +166,5 @@
   <!-- SC Port 1 -->
   <xacro:if value="$(arg sc_port_1_present)">
-    <xacro:sc_port prefix="sc_port_1" pose="${-0.075 + $(arg sc_port_1_translation)} 0.0705 0.0145 ${1.57 + $(arg sc_port_1_roll)} $(arg sc_port_1_pitch) ${1.57 + $(arg sc_port_1_yaw)}"/>
+    <xacro:sc_port prefix="sc_port_1" pose="${-0.075 + $(arg sc_port_1_translation)} 0.0705 0.0165 ${1.57 + $(arg sc_port_1_roll)} $(arg sc_port_1_pitch) ${1.57 + $(arg sc_port_1_yaw)}"/>
     <gazebo>
       <joint name="sc_port_1_joint" type="fixed">
@@ -176,5 +176,5 @@
   <!-- NIC Card Mount 0 (left-most) -->
   <xacro:if value="$(arg nic_card_mount_0_present)">
-    <xacro:nic_card_mount prefix="nic_card_mount_0" pose="${-0.081418 + $(arg nic_card_mount_0_translation)} -0.1745 0.01 $(arg nic_card_mount_0_roll) $(arg nic_card_mount_0_pitch) $(arg nic_card_mount_0_yaw)"/>
+    <xacro:nic_card_mount prefix="nic_card_mount_0" pose="${-0.081418 + $(arg nic_card_mount_0_translation)} -0.1745 0.012 $(arg nic_card_mount_0_roll) $(arg nic_card_mount_0_pitch) $(arg nic_card_mount_0_yaw)"/>
     <gazebo>
       <joint name="nic_card_mount_0_joint" type="fixed">
@@ -186,5 +186,5 @@
   <!-- NIC Card Mount 1 -->
   <xacro:if value="$(arg nic_card_mount_1_present)">
-    <xacro:nic_card_mount prefix="nic_card_mount_1" pose="${-0.081418 + $(arg nic_card_mount_1_translation)} -0.1345 0.01 $(arg nic_card_mount_1_roll) $(arg nic_card_mount_1_pitch) $(arg nic_card_mount_1_yaw)"/>
+    <xacro:nic_card_mount prefix="nic_card_mount_1" pose="${-0.081418 + $(arg nic_card_mount_1_translation)} -0.1345 0.012 $(arg nic_card_mount_1_roll) $(arg nic_card_mount_1_pitch) $(arg nic_card_mount_1_yaw)"/>
     <gazebo>
       <joint name="nic_card_mount_1_joint" type="fixed">
@@ -196,5 +196,5 @@
   <!-- NIC Card Mount 2 (center) -->
   <xacro:if value="$(arg nic_card_mount_2_present)">
-    <xacro:nic_card_mount prefix="nic_card_mount_2" pose="${-0.081418 + $(arg nic_card_mount_2_translation)} -0.0945 0.01 $(arg nic_card_mount_2_roll) $(arg nic_card_mount_2_pitch) $(arg nic_card_mount_2_yaw)"/>
+    <xacro:nic_card_mount prefix="nic_card_mount_2" pose="${-0.081418 + $(arg nic_card_mount_2_translation)} -0.0945 0.012 $(arg nic_card_mount_2_roll) $(arg nic_card_mount_2_pitch) $(arg nic_card_mount_2_yaw)"/>
     <gazebo>
       <joint name="nic_card_mount_2_joint" type="fixed">
@@ -206,5 +206,5 @@
   <!-- NIC Card Mount 3 -->
   <xacro:if value="$(arg nic_card_mount_3_present)">
-    <xacro:nic_card_mount prefix="nic_card_mount_3" pose="${-0.081418 + $(arg nic_card_mount_3_translation)} -0.0545 0.01 $(arg nic_card_mount_3_roll) $(arg nic_card_mount_3_pitch) $(arg nic_card_mount_3_yaw)"/>
+    <xacro:nic_card_mount prefix="nic_card_mount_3" pose="${-0.081418 + $(arg nic_card_mount_3_translation)} -0.0545 0.012 $(arg nic_card_mount_3_roll) $(arg nic_card_mount_3_pitch) $(arg nic_card_mount_3_yaw)"/>
     <gazebo>
       <joint name="nic_card_mount_3_joint" type="fixed">
@@ -216,5 +216,5 @@
   <!-- NIC Card Mount 4 (right-most) -->
   <xacro:if value="$(arg nic_card_mount_4_present)">
-    <xacro:nic_card_mount prefix="nic_card_mount_4" pose="${-0.081418 + $(arg nic_card_mount_4_translation)} -0.0145 0.01 $(arg nic_card_mount_4_roll) $(arg nic_card_mount_4_pitch) $(arg nic_card_mount_4_yaw)"/>
+    <xacro:nic_card_mount prefix="nic_card_mount_4" pose="${-0.081418 + $(arg nic_card_mount_4_translation)} -0.0145 0.012 $(arg nic_card_mount_4_roll) $(arg nic_card_mount_4_pitch) $(arg nic_card_mount_4_yaw)"/>
     <gazebo>
       <joint name="nic_card_mount_4_joint" type="fixed">
